File: Main Board v2.0/Kicad/ExpansionBus.kicad_sch (KiCad schematic)
At the start: 1 part, among them J1 Bus_ISA_16bit

Commit message: board update
Connections:
- net BC6 is gone; now on net MA22: J1.86 (LA19)
- net MA25 is gone; now on net MA21: J1.87 (LA18)
- net A12: now also J1.65 (IRQ10); no longer J1.50 (BA12)
- net A13: now also J1.66 (IRQ11); no longer J1.65 (IRQ10)
- net A14: now also J1.67 (IRQ12); no longer J1.66 (IRQ11)
- net A15: now also J1.68 (IRQ15); no longer J1.67 (IRQ12)
- net BINTACK0: now also J1.21 (IRQ7); no longer J1.68 (IRQ15)
- net BINTACK1: now also J1.22 (IRQ6); no longer J1.69 (IRQ14)
- net BINTACK2: now also J1.23 (IRQ5); no longer J1.70 (~{DACK0})
- net BINTACK3: now also J1.6 (DRQ2); no longer J1.71 (DRQ0)
- net BINTACK4: now also J1.8 (UNUSED); no longer J1.72 (~{DACK5})
- net BINTACK5: now also J1.72 (~{DACK5}); no longer J1.73 (DRQ5)
- net BINTACK7: now also J1.76 (~{DACK7}); no longer J1.75 (DRQ6)
- net BIRQ5: now also J1.73 (DRQ5); no longer J1.23 (IRQ5)
- net BIRQ6: now also J1.75 (DRQ6); no longer J1.22 (IRQ6)
- net BIRQ7: now also J1.77 (DRQ7); no longer J1.21 (IRQ7)
- net MA20: now also J1.88 (LA17); no longer J1.85 (LA20)
- net MA21: no longer J1.84 (LA21)
- net MA22: no longer J1.83 (LA22)
- net MA23: now also J1.85 (LA20); no longer J1.82 (LA23)
- net MA24: now also J1.84 (LA21); no longer J1.88 (LA17)
- new net BC2: J1.82 (LA23)
- new net BC3: J1.83 (LA22)
- new net MA12: J1.50 (BA12)
- no-connect marks 5 -> 4
Changed lines of the file:
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@@
 	(text "What is the max thickness of PCB that fits into ISA slot?\nThis seems to be 1.6mm."
 		(exclude_from_sim no)
-		(at 230.632 104.648 0)
+		(at 234.188 27.178 0)
 		(effects
 			(font
@@
 	)
 	(no_connect
-		(at 86.36 143.51)
+		(at 86.36 125.73)
 	)
 	(no_connect
-		(at 86.36 39.37)
+		(at 86.36 128.27)
 	)
 	(no_connect
-		(at 86.36 140.97)
-	)
-	(no_connect
-		(at 86.36 44.45)
+		(at 86.36 123.19)
 	)
 	(bus_entry
@@
 	)
 	(label "A13"
-		(at 86.36 113.03 0)
+		(at 86.36 115.57 0)
 		(effects
 			(font
@@
 	)
 	(label "MA22"
-		(at 160.02 113.03 180)
+		(at 160.02 120.65 180)
 		(effects
 			(font
@@
 		)
 	)
-	(label "MA25"
-		(at 44.45 31.75 180)
+	(label "A12"
+		(at 86.36 113.03 0)
 		(effects
 			(font
 				(size 1.27 1.27)
 			)
-			(justify right bottom)
+			(justify left bottom)
 		)
 	)
@@
 	)
 	(label "MA15"
-		(at 44.45 57.15 180)
+		(at 44.45 54.61 180)
 		(effects
 			(font
@@
 	)
 	(label "MA24"
-		(at 44.45 34.29 180)
+		(at 44.45 31.75 180)
 		(effects
 			(font
@@
 	)
 	(label "MA21"
-		(at 160.02 115.57 180)
+		(at 160.02 123.19 180)
 		(effects
 			(font
@@
 	)
 	(label "MA20"
-		(at 44.45 44.45 180)
+		(at 44.45 41.91 180)
 		(effects
 			(font
@@
 	)
 	(label "MA23"
-		(at 160.02 110.49 180)
+		(at 160.02 118.11 180)
 		(effects
 			(font
@@
 	)
 	(label "MA13"
-		(at 44.45 62.23 180)
+		(at 44.45 59.69 180)
 		(effects
 			(font
@@
 	)
 	(label "MA21"
-		(at 44.45 41.91 180)
+		(at 44.45 39.37 180)
 		(effects
 			(font
@@
 	)
 	(label "MA16"
-		(at 44.45 54.61 180)
+		(at 44.45 52.07 180)
 		(effects
 			(font
@@
 	)
 	(label "A14"
-		(at 86.36 115.57 0)
+		(at 86.36 118.11 0)
 		(effects
 			(font
@@
 	)
 	(label "MA20"
-		(at 160.02 118.11 180)
+		(at 160.02 125.73 180)
 		(effects
 			(font
@@
 		)
 	)
-	(label "A12"
+	(label "MA12"
 		(at 160.02 72.39 180)
 		(effects
@@
 	)
 	(label "A15"
-		(at 86.36 118.11 0)
+		(at 86.36 120.65 0)
 		(effects
 			(font
@@
 		)
 	)
+	(label "MA12"
+		(at 44.45 62.23 180)
+		(effects
+			(font
+				(size 1.27 1.27)
+			)
+			(justify right bottom)
+		)
+	)
 	(label "A4"
 		(at 160.02 92.71 180)
@@
 	)
 	(label "MA14"
-		(at 44.45 59.69 180)
+		(at 44.45 57.15 180)
 		(effects
 			(font
@@
 	)
 	(label "MA17"
-		(at 44.45 52.07 180)
+		(at 44.45 49.53 180)
 		(effects
 			(font
@@
 	)
 	(label "MA22"
-		(at 44.45 39.37 180)
+		(at 44.45 36.83 180)
 		(effects
 			(font
@@
 		)
 	)
-	(label "MA25"
-		(at 160.02 123.19 180)
-		(effects
-			(font
-				(size 1.27 1.27)
-			)
-			(justify right bottom)
-		)
-	)
 	(label "MA15"
 		(at 160.02 64.77 180)
@@
 	)
 	(label "MA23"
-		(at 44.45 36.83 180)
+		(at 44.45 34.29 180)
 		(effects
 			(font
@@
 	)
 	(label "MA18"
-		(at 44.45 49.53 180)
+		(at 44.45 46.99 180)
 		(effects
 			(font
@@
 	)
 	(label "MA24"
-		(at 160.02 125.73 180)
+		(at 160.02 115.57 180)
 		(effects
 			(font
@@
 	)
 	(label "MA19"
-		(at 44.45 46.99 180)
+		(at 44.45 44.45 180)
 		(effects
 			(font
@@
 		)
 	)
-	(global_label "BC6"
+	(global_label "BC2"
 		(shape input)
-		(at 160.02 120.65 0)
+		(at 160.02 110.49 0)
 		(fields_autoplaced yes)
 		(effects
@@
 		)
 		(property "Intersheetrefs" "${INTERSHEET_REFS}"
-			(at 166.7547 120.65 0)
+			(at 166.7547 110.49 0)
 			(hide yes)
 			(show_name no)
@@
 	(global_label "BINTACK4"
 		(shape input)
-		(at 86.36 130.81 180)
+		(at 86.36 44.45 180)
 		(fields_autoplaced yes)
 		(effects
@@
 		)
 		(property "Intersheetrefs" "${INTERSHEET_REFS}"
-			(at 74.3638 130.81 0)
+			(at 74.3638 44.45 0)
 			(hide yes)
 			(show_name no)
@@
 	(global_label "BINTACK2"
 		(shape input)
-		(at 86.36 125.73 180)
+		(at 86.36 82.55 180)
 		(fields_autoplaced yes)
 		(effects
@@
 		)
 		(property "Intersheetrefs" "${INTERSHEET_REFS}"
-			(at 74.3638 125.73 0)
+			(at 74.3638 82.55 0)
 			(hide yes)
 			(show_name no)
@@
 	(global_label "BINTACK5"
 		(shape input)
-		(at 86.36 133.35 180)
+		(at 86.36 130.81 180)
 		(fields_autoplaced yes)
 		(effects
@@
 		)
 		(property "Intersheetrefs" "${INTERSHEET_REFS}"
-			(at 74.3638 133.35 0)
+			(at 74.3638 130.81 0)
 			(hide yes)
 			(show_name no)
@@
 	(global_label "BINTACK3"
 		(shape input)
-		(at 86.36 128.27 180)
+		(at 86.36 39.37 180)
 		(fields_autoplaced yes)
 		(effects
@@
 		)
 		(property "Intersheetrefs" "${INTERSHEET_REFS}"
-			(at 74.3638 128.27 0)
+			(at 74.3638 39.37 0)
 			(hide yes)
 			(show_name no)
@@
 	(global_label "BIRQ5"
 		(shape input)
-		(at 86.36 82.55 180)
+		(at 86.36 133.35 180)
 		(fields_autoplaced yes)
 		(effects
@@
 		)
 		(property "Intersheetrefs" "${INTERSHEET_REFS}"
-			(at 77.69 82.55 0)
+			(at 77.69 133.35 0)
 			(hide yes)
 			(show_name no)
@@
 	(global_label "BIRQ7"
 		(shape input)
-		(at 86.36 77.47 180)
+		(at 86.36 143.51 180)
 		(fields_autoplaced yes)
 		(effects
@@
 		)
 		(property "Intersheetrefs" "${INTERSHEET_REFS}"
-			(at 77.69 77.47 0)
+			(at 77.69 143.51 0)
 			(hide yes)
 			(show_name no)
@@
 	(global_label "BIRQ6"
 		(shape input)
-		(at 86.36 80.01 180)
+		(at 86.36 138.43 180)
 		(fields_autoplaced yes)
 		(effects
@@
 		)
 		(property "Intersheetrefs" "${INTERSHEET_REFS}"
-			(at 77.69 80.01 0)
+			(at 77.69 138.43 0)
 			(hide yes)
 			(show_name no)
@@
 		)
 	)
+	(global_label "BC3"
+		(shape input)
+		(at 160.02 113.03 0)
+		(fields_autoplaced yes)
+		(effects
+			(font
+				(size 1.27 1.27)
+			)
+			(justify left)
+		)
+		(property "Intersheetrefs" "${INTERSHEET_REFS}"
+			(at 166.7547 113.03 0)
+			(hide yes)
+			(show_name no)
+			(do_not_autoplace no)
+			(effects
+				(font
+					(size 1.27 1.27)
+				)
+				(justify left)
+			)
+		)
+	)
 	(global_label "~{CPU_WR}"
 		(shape input)
@@
 	(global_label "BINTACK7"
 		(shape input)
-		(at 86.36 138.43 180)
+		(at 86.36 140.97 180)
 		(fields_autoplaced yes)
 		(effects
@@
 		)
 		(property "Intersheetrefs" "${INTERSHEET_REFS}"
-			(at 74.3638 138.43 0)
+			(at 74.3638 140.97 0)
 			(hide yes)
 			(show_name no)
@@
 	(global_label "BINTACK0"
 		(shape input)
-		(at 86.36 120.65 180)
+		(at 86.36 77.47 180)
 		(fields_autoplaced yes)
 		(effects
@@
 		)
 		(property "Intersheetrefs" "${INTERSHEET_REFS}"
-			(at 74.3638 120.65 0)
+			(at 74.3638 77.47 0)
 			(hide yes)
 			(show_name no)
@@
 	(global_label "BINTACK1"
 		(shape input)
-		(at 86.36 123.19 180)
+		(at 86.36 80.01 180)
 		(fields_autoplaced yes)
 		(effects
@@
 		)
 		(property "Intersheetrefs" "${INTERSHEET_REFS}"
-			(at 74.3638 123.19 0)
+			(at 74.3638 80.01 0)
 			(hide yes)
 			(show_name no)
@@
 		)
 	)
-	(hierarchical_label "MA[13..25]"
+	(hierarchical_label "MA[12..24]"
 		(shape input)
 		(at 25.4 25.4 180)

Commit message: board update
Connections:
- net BA1 is gone; now on net ~{CPU_WAIT}: J1.32 (IO)
- net BB4 is gone; now on net ~{CPU_M1}: J1.4 (IRQ2)
- net MA20: now also J1.42 (AEN); no longer J1.88 (LA17)
- net MA21: now also J1.41 (IO_READY); no longer J1.87 (LA18)
- net MA22: now also J1.88 (LA17); no longer J1.86 (LA19)
- net MA23: now also J1.87 (LA18); no longer J1.85 (LA20)
- net MA24: now also J1.86 (LA19); no longer J1.84 (LA21)
- net ~{CPU_M1}: no longer J1.42 (AEN)
- net ~{CPU_WAIT}: no longer J1.41 (IO_READY)
- new net BC4: J1.84 (LA21)
- new net BC5: J1.85 (LA20)
