File: Main Board v2.0/Kicad/Control Logic.kicad_sch (KiCad schematic)
At the start: 1 part, among them U8 XC95288XL-TQ144

Commit message: update
Parts:
- added C14, C15, C16, C17, C18, C19, C20, C21, C22, C23: 100n, symbol Device:C
- added J2: JTAG, symbol Connector_Generic:Conn_02x07_Odd_Even
- added R10, R11, R12: 4k7, symbol Device:R_Small
- added R6, R7, R8, R9: 100, symbol Device:R_Small
Connections:
- net +3V3: now reaches U8.1 (VCCIO)
- net +3V3: now also U8.109 (VCCIO), U8.127 (VCCIO), U8.141 (VCCINT), U8.37 (VCCIO), U8.42 (VCCINT), U8.55 (VCCIO), U8.73 (VCCIO), U8.8 (VCCINT), U8.84 (VCCINT), C14.1, C15.1, C16.1, C17.1, C18.1, C19.1, C20.1, C21.1, C22.1, C23.1, J2.1 (Pin_1), R10.2, R11.2, R12.2
- net D6: now reaches U8.10 (P10)
- net MROM_SEL0: now reaches U8.102 (P102)
- net MROM_SEL1: now reaches U8.103 (P103)
- net MROM_SEL2: now reaches U8.104 (P104)
- net MROM_SEL3: now reaches U8.105 (P105)
- net MMU_RAM1_DDIR: now reaches U8.106 (P106)
- net MROM_SEL4: now reaches U8.107 (P107)
- net GND: now reaches U8.108 (GND)
- net GND: now also U8.114 (GND), U8.123 (GND), U8.144 (GND), U8.18 (GND), U8.29 (GND), U8.36 (GND), U8.47 (GND), U8.62 (GND), U8.72 (GND), U8.89 (GND), U8.90 (GND), U8.99 (GND), C14.2, C15.2, C16.2, C17.2, C18.2, C19.2, C20.2, C21.2, C22.2, C23.2, J2.11 (Pin_11), J2.13 (Pin_13), J2.2 (Pin_2), J2.3 (Pin_3), J2.5 (Pin_5), J2.7 (Pin_7), J2.9 (Pin_9)
- net D7: now reaches U8.11 (P11)
- net ~{MMU_RAM1_DE}: now reaches U8.110 (P110)
- net MMU_RAM2_DDIR: now reaches U8.111 (P111)
- net ~{MMU_RAM2_DE}: now reaches U8.112 (P112)
- net MA20: now reaches U8.118 (P118)
- net ~{RESET}: now reaches U8.12 (P12)
- net at U8.122 (TDO): now also R8.1
- net MA21: now reaches U8.126 (P126)
- net MA22: now reaches U8.128 (P128)
- net MA23: now reaches U8.129 (P129)
- net ~{NMI}: now reaches U8.13 (P13)
- net MA24: now reaches U8.130 (P130)
- net MA25: now reaches U8.131 (P131)
- net MA26: now reaches U8.132 (P132)
- net MA27: now reaches U8.133 (P133)
- net MA28: now reaches U8.134 (P134)
- net ~{ME0}: now reaches U8.135 (P135)
- net ~{ME1}: now reaches U8.136 (P136)
- net ~{ME2}: now reaches U8.137 (P137)
- net ~{ME3}: now reaches U8.138 (P138)
- net ~{ME4}: now reaches U8.139 (P139)
- net ~{INT}: now reaches U8.14 (P14)
- net ~{RFSH}: now reaches U8.142 (P142)
- net ~{WAIT}: now reaches U8.143 (I/O/GSR)
- net ~{M1}: now reaches U8.15 (P15)
- net A0: now reaches U8.16 (P16)
- net A1: now reaches U8.17 (P17)
- net A2: now reaches U8.19 (P19)
- net A15: now reaches U8.2 (I/O/GTS3)
- net A3: now reaches U8.20 (P20)
- net A4: now reaches U8.21 (P21)
- net A5: now reaches U8.22 (P22)
- net A6: now reaches U8.23 (P23)
- net A7: now reaches U8.24 (P24)
- net A8: now reaches U8.25 (P25)
- net A9: now reaches U8.26 (P26)
- net A10: now reaches U8.27 (P27)
- net A11: now reaches U8.28 (P28)
- net D0: now reaches U8.3 (I/O/GTS4)
- net A12: now reaches U8.30 (I/O/GCK1)
- net A13: now reaches U8.31 (P31)
- net CLK20: now reaches U8.32 (I/O/GCK2)
- net ~{HALT}: now reaches U8.33 (P33)
- net ~{RD}: now reaches U8.34 (P34)
- net A14: now reaches U8.35 (P35)
- net ~{WR}: now reaches U8.38 (I/O/GCK3)
- net ~{MREQ}: now reaches U8.39 (P39)
- net D1: now reaches U8.4 (P4)
- net ~{IORQ}: now reaches U8.40 (P40)
- net ~{BUSRQ}: now reaches U8.41 (P41)
- net ~{BUSACK}: now reaches U8.43 (P43)
- net MA13: now reaches U8.44 (P44)
- net MA14: now reaches U8.45 (P45)
- net MA15: now reaches U8.46 (P46)
- net MA16: now reaches U8.48 (P48)
- net MA17: now reaches U8.49 (P49)
- net D2: now reaches U8.5 (I/O/GTS1)
- net MA18: now reaches U8.50 (P50)
- net MA19: now reaches U8.51 (P51)
- net MMU_MEML_CP: now reaches U8.52 (P52)
- net MMU_MEML_OE: now reaches U8.53 (P53)
- net MMU_IOL_CP: now reaches U8.54 (P54)
- net MMU_IOL_OE: now reaches U8.56 (P56)
- net MMU_MAP_SEL0: now reaches U8.57 (P57)
- net MMU_MAP_SEL1: now reaches U8.58 (P58)
- net MMU_MAP_SEL2: now reaches U8.59 (P59)
- net D3: now reaches U8.6 (I/O/GTS2)
- net MMU_MAP_SEL3: now reaches U8.60 (P60)
- net ~{MMU_RAM1_CE}: now reaches U8.61 (P61)
- net at U8.63 (TDI): now also R7.1
- net ~{MMU_RAM1_OE}: now reaches U8.64 (P64)
- net at U8.65 (TMS): now also R9.1
- net ~{MMU_RAM1_WE}: now reaches U8.66 (P66)
- net at U8.67 (TCK): now also R6.1
- net ~{MMU_RAM2_CE}: now reaches U8.68 (P68)
- net ~{MMU_RAM2_OE}: now reaches U8.69 (P69)
- net D4: now reaches U8.7 (P7)
- net ~{MMU_RAM2_WE}: now reaches U8.70 (P70)
- net D5: now reaches U8.9 (P9)
- new net INIT: J2.14 (Pin_14)
- new net TCK: J2.6 (Pin_6), R11.1, R6.2
- new net TDI: J2.10 (Pin_10), R12.1, R7.2
- new net TDO: J2.8 (Pin_8), R8.2
- new net TMS: J2.4 (Pin_4), R10.1, R9.2
- no-connect marks 0 -> 1
Other:
- note added: "12 signals"
- note added: "16 signals"
- note added: "18 signals"
- note added: "38 signals"
- note added: "ALT: 22 signals"
- note added: "https://pcbsync.com/xilinx-jtagdebug/"

Commit message: schematic done*
Parts:
- added C19: 100n, Capacitor_SMD:C_0603_1608Metric_Pad1.08x0.95mm_HandSolder, symbol Device:C_Small
- added C20, C21: 100u, symbol Device:C_Polarized_Small
- added J4: +3V3 Supply, Connector_PinHeader_2.54mm:PinHeader_1x01_P2.54mm_Vertical, symbol Connector:Conn_01x01_Pin
- added J5: Unused CPLD Signals, Connector_PinHeader_2.54mm:PinHeader_2x20_P2.54mm_Vertical, symbol Connector_Generic:Conn_02x20_Odd_Even
- added U8: AP1117-33, Package_TO_SOT_SMD:SOT-223-3_TabPin2, symbol Regulator_Linear:AP1117-33
- C10: renamed from C15; footprint (none) -> Capacitor_SMD:C_0603_1608Metric_Pad1.08x0.95mm_HandSolder
- C11: renamed from C16; footprint (none) -> Capacitor_SMD:C_0603_1608Metric_Pad1.08x0.95mm_HandSolder
- C12: renamed from C17; footprint (none) -> Capacitor_SMD:C_0603_1608Metric_Pad1.08x0.95mm_HandSolder
- C13: renamed from C18; footprint (none) -> Capacitor_SMD:C_0603_1608Metric_Pad1.08x0.95mm_HandSolder
- C14: renamed from C19; footprint (none) -> Capacitor_SMD:C_0603_1608Metric_Pad1.08x0.95mm_HandSolder
- C15: renamed from C20; footprint (none) -> Capacitor_SMD:C_0603_1608Metric_Pad1.08x0.95mm_HandSolder
- C16: renamed from C21; footprint (none) -> Capacitor_SMD:C_0603_1608Metric_Pad1.08x0.95mm_HandSolder
- C17: renamed from C22; footprint (none) -> Capacitor_SMD:C_0603_1608Metric_Pad1.08x0.95mm_HandSolder
- C18: renamed from C23; footprint (none) -> Capacitor_SMD:C_0603_1608Metric_Pad1.08x0.95mm_HandSolder
- C9: renamed from C14; footprint (none) -> Capacitor_SMD:C_0603_1608Metric_Pad1.08x0.95mm_HandSolder
- J3: renamed from J2; footprint (none) -> Connector_PinHeader_2.54mm:PinHeader_2x07_P2.54mm_Vertical
- R2: renamed from R10; footprint (none) -> Resistor_SMD:R_0603_1608Metric_Pad0.98x0.95mm_HandSolder
- R3: renamed from R11; footprint (none) -> Resistor_SMD:R_0603_1608Metric_Pad0.98x0.95mm_HandSolder
- R4: renamed from R12; footprint (none) -> Resistor_SMD:R_0603_1608Metric_Pad0.98x0.95mm_HandSolder
- R5: renamed from R6; footprint (none) -> Resistor_SMD:R_0603_1608Metric_Pad0.98x0.95mm_HandSolder
- R6: renamed from R7; footprint (none) -> Resistor_SMD:R_0603_1608Metric_Pad0.98x0.95mm_HandSolder
- R7: renamed from R8; footprint (none) -> Resistor_SMD:R_0603_1608Metric_Pad0.98x0.95mm_HandSolder
- R8: renamed from R9; footprint (none) -> Resistor_SMD:R_0603_1608Metric_Pad0.98x0.95mm_HandSolder
- renumbered U8 to U7
Connections:
- net +3V3: now also J3.2 (Pin_2), C19.1, C21.1, J4.1 (Pin_1), U8.2 (VO); no longer J3.1 (Pin_1)
- net BCLK: now also U7.71 (P71)
- net BIRQ2: now also U7.78 (P78)
- net BIRQ3: now also U7.79 (P79)
- net BIRQ4: now also U7.80 (P80)
- net BIRQ5: now also U7.81 (P81)
- net BIRQ6: now also U7.82 (P82)
- net BIRQ7: now also U7.83 (P83)
- net GND: now also J3.1 (Pin_1), C19.2, C20.2, C21.2, U8.1 (GND); no longer J3.2 (Pin_2)
- net MMU_RAM1_DDIR: now also U7.113 (P113); no longer U7.106 (P106)
- net MMU_RAM2_DDIR: now also U7.116 (P116); no longer U7.111 (P111)
- net ~{B8_MEM_RD}: now also U7.77 (P77)
- net ~{B8_MEM_WR}: now also U7.76 (P76)
- net ~{BIO_RD}: now also U7.75 (P75)
- net ~{BIO_WR}: now also U7.74 (P74)
- net ~{MMU_RAM1_CE}: now also U7.69 (P69); no longer U7.61 (P61)
- net ~{MMU_RAM1_DE}: now also U7.115 (P115); no longer U7.110 (P110)
- net ~{MMU_RAM1_OE}: now also U7.70 (P70); no longer U7.64 (P64)
- net ~{MMU_RAM1_WE}: now also U7.106 (P106); no longer U7.66 (P66)
- net ~{MMU_RAM2_CE}: now also U7.110 (P110); no longer U7.68 (P68)
- net ~{MMU_RAM2_DE}: now also U7.117 (P117); no longer U7.112 (P112)
- net ~{MMU_RAM2_OE}: now also U7.111 (P111); no longer U7.69 (P69)
- net ~{MMU_RAM2_WE}: now also U7.112 (P112); no longer U7.70 (P70)
- net CTRL21: now reaches U7.100 (P100)
- net CTRL21: now also J5.4 (Pin_4)
- net CTRL22: now reaches U7.101 (P101)
- net CTRL22: now also J5.6 (Pin_6)
- net CTRL4: now reaches U7.119 (P119)
- net CTRL4: now also J5.9 (Pin_9)
- net CTRL5: now reaches U7.120 (P120)
- net CTRL5: now also J5.11 (Pin_11)
- net CTRL6: now reaches U7.121 (P121)
- net CTRL6: now also J5.13 (Pin_13)
- net CTRL7: now reaches U7.124 (P124)
- net CTRL7: now also J5.15 (Pin_15)
- net CTRL8: now reaches U7.125 (P125)
- net CTRL8: now also J5.17 (Pin_17)
- net CTRL3: now reaches U7.140 (P140)
- net CTRL3: now also J5.7 (Pin_7)
- net CTRL9: now reaches U7.85 (P85)
- net CTRL9: now also J5.19 (Pin_19)
- net CTRL10: now reaches U7.86 (P86)
- net CTRL10: now also J5.21 (Pin_21)
- net CTRL11: now reaches U7.87 (P87)
- net CTRL11: now also J5.23 (Pin_23)
- net CTRL12: now reaches U7.88 (P88)
- net CTRL12: now also J5.25 (Pin_25)
- net CTRL13: now reaches U7.91 (P91)
- net CTRL13: now also J5.27 (Pin_27)
- net CTRL14: now reaches U7.92 (P92)
- net CTRL14: now also J5.29 (Pin_29)
- net CTRL15: now reaches U7.93 (P93)
- net CTRL15: now also J5.31 (Pin_31)
- net CTRL16: now reaches U7.94 (P94)
- net CTRL16: now also J5.33 (Pin_33)
- net CTRL17: now reaches U7.95 (P95)
- net CTRL17: now also J5.35 (Pin_35)
- net CTRL18: now reaches U7.96 (P96)
- net CTRL18: now also J5.37 (Pin_37)
- net CTRL19: now reaches U7.97 (P97)
- net CTRL19: now also J5.39 (Pin_39)
- net CTRL20: now reaches U7.98 (P98)
- net CTRL20: now also J5.2 (Pin_2)
- net INIT renamed HALT
- net MA26 renamed MMU_MP_RD
- net MA27 renamed MMU_MP_WR
- net MA28 renamed MMU_MP_EXE
- net MMU_IOL_CP renamed MMU_MAP2
- net MMU_IOL_OE renamed MMU_MAP3
- net MMU_MAP_SEL0 renamed MMU_MAP4
- net MMU_MAP_SEL1 renamed MMU_MAP5
- net MMU_MAP_SEL2 renamed MMU_MAP6
- net MMU_MAP_SEL3 renamed MMU_MAP7
- net MMU_MEML_CP renamed MMU_MAP0
- net MMU_MEML_OE renamed MMU_MAP1
- net MROM_SEL0 renamed CTRL23
- net CTRL23: now also J5.8 (Pin_8)
- net MROM_SEL1 renamed CTRL24
- net CTRL24: now also J5.10 (Pin_10)
- net MROM_SEL2 renamed CTRL25
- net CTRL25: now also J5.12 (Pin_12)
- net MROM_SEL3 renamed CTRL26
- net CTRL26: now also J5.14 (Pin_14)
- net MROM_SEL4 renamed CTRL27
- net CTRL27: now also J5.16 (Pin_16)
- net ~{BUSACK} renamed ~{CPU_BUSACK}
- net ~{BUSRQ} renamed ~{CPU_BUSRQ}
- net ~{HALT} renamed ~{CPU_HALT}
- net ~{INT} renamed ~{CPU_INT}
- net ~{IORQ} renamed ~{CPU_IORQ}
- net ~{M1} renamed ~{CPU_M1}
- net ~{ME0} renamed ~{ROM_CE}
- net ~{ME1} renamed ~{RAM_CE}
- net ~{ME2} renamed CTRL0
- net CTRL0: now also J5.1 (Pin_1)
- net ~{ME3} renamed CTRL1
- net CTRL1: now also J5.3 (Pin_3)
- net ~{ME4} renamed CTRL2
- net CTRL2: now also J5.5 (Pin_5)
- net ~{MREQ} renamed ~{CPU_MREQ}
- net ~{NMI} renamed ~{CPU_NMI}
- net ~{RD} renamed ~{CPU_RD}
- net ~{RESET} renamed ~{CPU_RST}
- net ~{RFSH} renamed ~{CPU_RFSH}
- net ~{WAIT} renamed ~{CPU_WAIT}
- net ~{WR} renamed ~{CPU_WR}
- new net +5V: C20.1, U8.3 (VI)
- new net MMU_MAP10: U7.66 (P66)
- new net MMU_MAP11: U7.68 (P68)
- new net MMU_MAP8: U7.61 (P61)
- new net MMU_MAP9: U7.64 (P64)
- no-connect marks 1 -> 14
Other:
- note added: "Optional +3V3 supply"
- note added: "Pin assignments are flexible. CLK20 must go on a GCKn pin."
- note removed: "12 signals"
- note removed: "16 signals"
- note removed: "18 signals"
- note removed: "38 signals"
- note removed: "ALT: 22 signals"
- note removed: "https://pcbsync.com/xilinx-jtagdebug/"
- moved on the sheet: J3, R2, R3, R4

Commit message: board update
Parts:
- removed J5: Unused CPLD Signals, Connector_PinHeader_2.54mm:PinHeader_2x20_P2.54mm_Vertical, symbol Connector_Generic:Conn_02x20_Odd_Even
- added J5: Conn_02x14_Counter_Clockwise, Connector_PinSocket_2.54mm:PinSocket_2x14_P2.54mm_Vertical, symbol Connector_Generic:Conn_02x14_Counter_Clockwise
- C20, C21: footprint (none) -> Capacitor_THT:CP_Radial_D10.0mm_P5.00mm
Connections:
- net CTRL25 is gone; now on net CTRL22: U7.104 (P104)
- net CTRL26 is gone; now on net CTRL23: U7.105 (P105)
- net CTRL27 is gone; now on net CTRL24: U7.107 (P107)
- net CTRL0: now also J5.1 (Pin_1)
- net CTRL1: now also J5.2 (Pin_2)
- net CTRL10: now also U7.91 (P91), J5.11 (Pin_11); no longer U7.86 (P86)
- net CTRL11: now also U7.92 (P92), J5.12 (Pin_12); no longer U7.87 (P87)
- net CTRL12: now also U7.93 (P93), J5.13 (Pin_13); no longer U7.88 (P88)
- net CTRL13: now also U7.94 (P94), J5.28 (Pin_28); no longer U7.91 (P91)
- net CTRL14: now also U7.95 (P95), J5.27 (Pin_27); no longer U7.92 (P92)
- net CTRL15: now also U7.96 (P96), J5.26 (Pin_26); no longer U7.93 (P93)
- net CTRL16: now also U7.97 (P97), J5.25 (Pin_25); no longer U7.94 (P94)
- net CTRL17: now also U7.98 (P98), J5.24 (Pin_24); no longer U7.95 (P95)
- net CTRL18: now also U7.100 (P100), J5.23 (Pin_23); no longer U7.96 (P96)
- net CTRL19: now also U7.101 (P101), J5.22 (Pin_22); no longer U7.97 (P97)
- net CTRL2: now also J5.3 (Pin_3)
- net CTRL20: now also U7.102 (P102), J5.21 (Pin_21); no longer U7.98 (P98)
- net CTRL21: now also U7.103 (P103), J5.20 (Pin_20); no longer U7.100 (P100)
- net CTRL22: now also J5.19 (Pin_19); no longer U7.101 (P101)
- net CTRL23: now also J5.18 (Pin_18); no longer U7.102 (P102)
- net CTRL24: now also J5.17 (Pin_17); no longer U7.103 (P103)
- net CTRL3: now also J5.4 (Pin_4)
- net CTRL4: now also U7.121 (P121), J5.5 (Pin_5); no longer U7.119 (P119)
- net CTRL5: now also U7.124 (P124), J5.6 (Pin_6); no longer U7.120 (P120)
- net CTRL6: now also U7.125 (P125), J5.7 (Pin_7); no longer U7.121 (P121)
- net CTRL7: now also U7.86 (P86), J5.8 (Pin_8); no longer U7.124 (P124)
- net CTRL8: now also U7.87 (P87), J5.9 (Pin_9); no longer U7.125 (P125)
- net CTRL9: now also U7.88 (P88), J5.10 (Pin_10); no longer U7.85 (P85)
- net MMU_RAM1_DDIR: now also U7.116 (P116); no longer U7.113 (P113)
- net MMU_RAM2_DDIR: now also U7.119 (P119); no longer U7.116 (P116)
- net ~{MMU_RAM1_CE}: now also U7.106 (P106); no longer U7.69 (P69)
- net ~{MMU_RAM1_DE}: now also U7.117 (P117); no longer U7.115 (P115)
- net ~{MMU_RAM1_OE}: now also U7.110 (P110); no longer U7.70 (P70)
- net ~{MMU_RAM1_WE}: now also U7.111 (P111); no longer U7.106 (P106)
- net ~{MMU_RAM2_CE}: now also U7.112 (P112); no longer U7.110 (P110)
- net ~{MMU_RAM2_DE}: now also U7.120 (P120); no longer U7.117 (P117)
- net ~{MMU_RAM2_OE}: now also U7.113 (P113); no longer U7.111 (P111)
- net ~{MMU_RAM2_WE}: now also U7.115 (P115); no longer U7.112 (P112)
- new net MMU_MAP12: U7.69 (P69)
- new net MMU_MAP13: U7.70 (P70)
- new net ~{BIACK}: U7.85 (P85)
- no-connect marks 14 -> 5
