File: Main Board v2.0/Kicad/Control Logic.kicad_sch (KiCad schematic)
At the start: 20 parts, among them J2 +3V3 Supply, J3 JTAG, U7 XC95288XL-TQ144, U8 AP1117-33

Commit message: board progress
Connections:
- net A12: now also U7.140 (P140); no longer U7.136 (P136)
- net A13: now also U7.139 (P139); no longer U7.137 (P137)
- net A15: now also U7.137 (P137); no longer U7.139 (P139)
- net BCLK: now also U7.126 (P126); no longer U7.83 (P83)
- net BINTACK1: now also U7.130 (P130); no longer U7.132 (P132)
- net BINTACK2: now also U7.131 (P131); no longer U7.85 (P85)
- net BINTACK3: now also U7.75 (P75); no longer U7.86 (P86)
- net BINTACK4: now also U7.74 (P74); no longer U7.87 (P87)
- net BINTEN: now also U7.85 (P85); no longer U7.79 (P79)
- net BIRQ0: now also U7.136 (P136); no longer U7.133 (P133)
- net BIRQ1: now also U7.135 (P135); no longer U7.134 (P134)
- net BIRQ2: now also U7.134 (P134); no longer U7.135 (P135)
- net BIRQ3: now also U7.133 (P133); no longer U7.140 (P140)
- net BIRQ4: now also U7.132 (P132); no longer U7.88 (P88)
- net SYSCMD: now also U7.82 (P82); no longer U7.124 (P124)
- net SYSDDIR: now also U7.86 (P86); no longer U7.120 (P120)
- net SYSINT0: now also U7.83 (P83); no longer U7.126 (P126)
- net SYSINT1: now also U7.81 (P81); no longer U7.128 (P128)
- net SYSINT2: now also U7.79 (P79); no longer U7.129 (P129)
- net SYSINTACK: now also U7.80 (P80); no longer U7.125 (P125)
- net ~{B8_MEM_RD}: now also U7.77 (P77); no longer U7.75 (P75)
- net ~{B8_MEM_WR}: now also U7.76 (P76); no longer U7.74 (P74)
- net ~{BIACK}: now also U7.121 (P121); no longer U7.78 (P78)
- net ~{BIO_RD}: now also U7.88 (P88); no longer U7.77 (P77)
- net ~{BIO_WR}: now also U7.78 (P78); no longer U7.76 (P76)
- net ~{CPU_BUSACK}: now also U7.128 (P128); no longer U7.81 (P81)
- net ~{CPU_BUSRQ}: now also U7.125 (P125); no longer U7.80 (P80)
- net ~{CPU_INT}: now also U7.120 (P120); no longer U7.131 (P131)
- net ~{CPU_NMI}: now also U7.129 (P129); no longer U7.130 (P130)
- net ~{CPU_RFSH}: now also U7.124 (P124); no longer U7.82 (P82)
- net ~{SYSDEN}: now also U7.87 (P87); no longer U7.121 (P121)
