File: Main Board v2.0/Kicad/Main Board v2.0.kicad_pcb (KiCad board)
At the start: 4 copper layers, 0 parts

Commit message: board update
Parts:
- added C1: 100n, Capacitor_SMD:C_0603_1608Metric_Pad1.08x0.95mm_HandSolder, F.Cu at (387.6, 168.4)
- added C10: 100n, Capacitor_SMD:C_0603_1608Metric_Pad1.08x0.95mm_HandSolder, F.Cu at (368.4, 120.8)
- added C11: 100n, Capacitor_SMD:C_0603_1608Metric_Pad1.08x0.95mm_HandSolder, F.Cu at (368.4, 123.3)
- added C12: 100n, Capacitor_SMD:C_0603_1608Metric_Pad1.08x0.95mm_HandSolder, F.Cu at (368.4, 125.8)
- added C13: 100n, Capacitor_SMD:C_0603_1608Metric_Pad1.08x0.95mm_HandSolder, F.Cu at (368.4, 128.3)
- added C14: 100n, Capacitor_SMD:C_0603_1608Metric_Pad1.08x0.95mm_HandSolder, F.Cu at (368.4, 130.9)
- added C15: 100n, Capacitor_SMD:C_0603_1608Metric_Pad1.08x0.95mm_HandSolder, F.Cu at (368.4, 133.4)
- added C16: 100n, Capacitor_SMD:C_0603_1608Metric_Pad1.08x0.95mm_HandSolder, F.Cu at (372.8, 118.3)
- added C17: 100n, Capacitor_SMD:C_0603_1608Metric_Pad1.08x0.95mm_HandSolder, F.Cu at (372.8, 120.8)
- added C18: 100n, Capacitor_SMD:C_0603_1608Metric_Pad1.08x0.95mm_HandSolder, F.Cu at (372.8, 123.3)
- added C19: 100n, Capacitor_SMD:C_0603_1608Metric_Pad1.08x0.95mm_HandSolder, F.Cu at (372.8, 125.8)
- added C2: 100n, Capacitor_SMD:C_0603_1608Metric_Pad1.08x0.95mm_HandSolder, F.Cu at (387.6, 170.9)
- added C20: 100u, Capacitor_THT:CP_Radial_D10.0mm_P5.00mm, F.Cu at (251.3, 99.8)
- added C21: 100u, Capacitor_THT:CP_Radial_D10.0mm_P5.00mm, F.Cu at (251.3, 111.3)
- added C22: 100n, Capacitor_SMD:C_0201_0603Metric_Pad0.64x0.40mm_HandSolder, F.Cu at (406.2, 112.0)
- added C23: 100n, Capacitor_SMD:C_0201_0603Metric_Pad0.64x0.40mm_HandSolder, F.Cu at (406.2, 113.7)
- added C24: 100u, Capacitor_THT:CP_Radial_D10.0mm_P5.00mm, F.Cu at (265.1, 99.8)
- added C3: 100n, Capacitor_SMD:C_0603_1608Metric_Pad1.08x0.95mm_HandSolder, F.Cu at (387.6, 173.4)
- added C4: 100n, Capacitor_SMD:C_0603_1608Metric_Pad1.08x0.95mm_HandSolder, F.Cu at (387.6, 175.9)
- added C5: 100n, Capacitor_SMD:C_0603_1608Metric_Pad1.08x0.95mm_HandSolder, F.Cu at (387.6, 178.4)
- added C6: 100n, Capacitor_SMD:C_0603_1608Metric_Pad1.08x0.95mm_HandSolder, F.Cu at (387.6, 181.0)
- added C7: 100n, Capacitor_SMD:C_0603_1608Metric_Pad1.08x0.95mm_HandSolder, F.Cu at (335.4, 116.1)
- added C8: 100n, Capacitor_SMD:C_0603_1608Metric_Pad1.08x0.95mm_HandSolder, F.Cu at (335.4, 118.6)
- added C9: 100n, Capacitor_SMD:C_0603_1608Metric_Pad1.08x0.95mm_HandSolder, F.Cu at (368.4, 118.3)
- added J1: Bus_ISA_16bit, Connector_PCBEdge:BUS_AT, F.Cu at (210.1, 130.8)
- added J2: Conn_02x20_Odd_Even, Connector_PinSocket_2.54mm:PinSocket_2x20_P2.54mm_Vertical, F.Cu at (151.5, 120.9)
- added J3: JTAG, Connector_PinHeader_2.54mm:PinHeader_2x07_P2.54mm_Vertical, F.Cu at (187.6, 115.6)
- added J4: +3V3 Supply, Connector_PinHeader_2.54mm:PinHeader_1x01_P2.54mm_Vertical, F.Cu at (178.2, 99.6)
- added J5: Conn_02x14_Counter_Clockwise, Connector_PinSocket_2.54mm:PinSocket_2x14_P2.54mm_Vertical, F.Cu at (222.4, 75.1)
- added R2: 4k7, Resistor_SMD:R_0603_1608Metric_Pad0.98x0.95mm_HandSolder, F.Cu at (372.8, 128.3)
- added R3: 4k7, Resistor_SMD:R_0603_1608Metric_Pad0.98x0.95mm_HandSolder, F.Cu at (372.8, 130.9)
- added R4: 4k7, Resistor_SMD:R_0603_1608Metric_Pad0.98x0.95mm_HandSolder, F.Cu at (372.8, 133.4)
- added R5: 100, Resistor_SMD:R_0603_1608Metric_Pad0.98x0.95mm_HandSolder, F.Cu at (377.1, 118.3)
- added R6: 100, Resistor_SMD:R_0603_1608Metric_Pad0.98x0.95mm_HandSolder, F.Cu at (377.1, 120.8)
- added R7: 100, Resistor_SMD:R_0603_1608Metric_Pad0.98x0.95mm_HandSolder, F.Cu at (377.1, 123.3)
- added R8: 100, Resistor_SMD:R_0603_1608Metric_Pad0.98x0.95mm_HandSolder, F.Cu at (377.1, 125.8)
- added RN1: 10k, Resistor_THT:R_Array_SIP9, F.Cu at (130.0, 91.1)
- added U10: CY7C109B, Package_SO:SOJ-32_10.16x20.955mm_P1.27mm, F.Cu at (186.8, 65.3)
- added U11: CY7C109B, Package_SO:SOJ-32_10.16x20.955mm_P1.27mm, F.Cu at (200.4, 65.3)
- added U3: 74HCT245, Package_DIP:CERDIP-20_W7.62mm_SideBrazed_LongPads_Socket, F.Cu at (157.0, 54.4)
- added U4: 74HCT245, Package_DIP:CERDIP-20_W7.62mm_SideBrazed_LongPads_Socket, F.Cu at (169.3, 54.4)
- added U5: AS6C4008-55PCN, Package_SO:SOP-32_11.305x20.495mm_P1.27mm, F.Cu at (142.5, 74.0)
- added U6: AM29F040B, Socket:3M_Textool_232-1288-00-0602J_2x16_P2.54mm, F.Cu at (107.4, 51.6)
- added U7: XC95288XL-TQ144, Package_QFP:TQFP-144_20x20mm_P0.5mm, F.Cu at (193.9, 93.0)
- added U8: AP1117-33, Package_TO_SOT_SMD:SOT-223-3_TabPin2, F.Cu at (173.6, 109.5)
- added U9: Z80CPU, Socket:3M_Textool_240-1288-00-0602J_2x20_P2.54mm, F.Cu at (81.0, 51.6)
- added Y1: 20MHz, Oscillator:Oscillator_DIP-14, F.Cu at (96.9, 112.0)

Commit message: schematic update
Parts:
- added J10: SPI, Connector_PinSocket_2.54mm:PinSocket_2x03_P2.54mm_Vertical, F.Cu at (261.7, 39.6)
- added J6: AVR-JTAG-10, Connector_IDC:IDC-Header_2x05_P2.54mm_Vertical, F.Cu at (259.6, 61.3)
- added J7: USART0, Connector_PinHeader_2.54mm:PinHeader_1x04_P2.54mm_Vertical, F.Cu at (259.2, 27.4)
- added J8: USART1, Connector_PinHeader_2.54mm:PinHeader_1x04_P2.54mm_Vertical, F.Cu at (263.8, 27.4)
- added J9: PS2KB, Connector_PinHeader_2.54mm:PinHeader_1x04_P2.54mm_Vertical, F.Cu at (268.4, 27.4)
- added U1: GLT725608, Package_SO:SOJ-28_7.62x18.415mm_P1.27mm, F.Cu at (190.4, 59.2)
- added U2: GLT725608, Package_SO:SOJ-28_7.62x18.415mm_P1.27mm, F.Cu at (201.3, 59.2)
- C20, C21, C24: footprint Capacitor_THT:CP_Radial_D10.0mm_P5.00mm -> Capacitor_THT:CP_Radial_D8.0mm_P3.80mm
- J2: value Conn_02x20_Odd_Even -> Spare Extension Bus Signals
- J3: footprint Connector_PinHeader_2.54mm:PinHeader_2x07_P2.54mm_Vertical -> Connector_IDC:IDC-Header_2x07_P2.54mm_Vertical
- J5: value Conn_02x14_Counter_Clockwise -> Conn_02x10_Odd_Even; footprint Connector_PinSocket_2.54mm:PinSocket_2x14_P2.54mm_Vertical -> Connector_PinSocket_2.54mm:PinSocket_2x10_P2.54mm_Vertical
- U10: value CY7C109B -> ATmega1284-P; footprint Package_SO:SOJ-32_10.16x20.955mm_P1.27mm -> Package_DIP:DIP-40_W15.24mm
- U11: value CY7C109B -> 74HCT245; footprint Package_SO:SOJ-32_10.16x20.955mm_P1.27mm -> Package_DIP:DIP-20_W7.62mm_Socket_LongPads
- moved C1 285.4 mm to (140.1, 26.3)
- moved C2 285.4 mm to (140.1, 28.8)
- moved C3 285.4 mm to (140.1, 31.3)
- moved C4 285.4 mm to (140.1, 33.8)
- moved C5 285.4 mm to (140.1, 36.4)
- moved C6 285.4 mm to (140.1, 38.9)
- moved C22 141.5 mm to (267.7, 140.6)
- moved C23 141.5 mm to (267.7, 142.4)
- moved C16 141.5 mm to (234.2, 146.9)
- moved C17 141.5 mm to (234.2, 149.4)
- moved C18 141.5 mm to (234.2, 151.9)
- moved C19 141.5 mm to (234.2, 154.5)
- moved R2 141.5 mm to (234.2, 157.0)
- moved R3 141.5 mm to (234.2, 159.5)
- moved R4 141.5 mm to (234.2, 162.0)
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Connections:
- J1 pad 28: /Expansion Bus/BB28 -> BINTEN
- J1 pad 65: /Expansion Bus/BD3 -> /CPU/A13
- J1 pad 66: /Expansion Bus/BD4 -> /CPU/A14
- J1 pad 67: /Expansion Bus/BD5 -> /CPU/A15
- J2 pad 11: /Expansion Bus/BB28 -> unconnected-(J2-Pin_11-Pad11)
- J2 pad 13: /Expansion Bus/BD3 -> unconnected-(J2-Pin_13-Pad13)
- J2 pad 15: /Expansion Bus/BD4 -> unconnected-(J2-Pin_15-Pad15)
- J2 pad 17: /Expansion Bus/BD5 -> unconnected-(J2-Pin_17-Pad17)
- J5 pad 10: /Control Logic/CTRL9 -> /Control Logic/CTRL21
- J5 pad 11: /Control Logic/CTRL10 -> /Control Logic/CTRL5
- J5 pad 12: /Control Logic/CTRL11 -> /Control Logic/CTRL22
- J5 pad 13: /Control Logic/CTRL12 -> /Control Logic/CTRL6
- J5 pad 14: unconnected-(J5-Pin_14-Pad14) -> /Control Logic/CTRL23
- J5 pad 15: unconnected-(J5-Pin_15-Pad15) -> /Control Logic/CTRL7
- J5 pad 16: unconnected-(J5-Pin_16-Pad16) -> /Control Logic/CTRL24
- J5 pad 17: /Control Logic/CTRL24 -> /Control Logic/CTRL8
- J5 pad 18: /Control Logic/CTRL23 -> /Control Logic/CTRL25
- J5 pad 19: /Control Logic/CTRL22 -> /Control Logic/CTRL9
- J5 pad 2: /Control Logic/CTRL1 -> /Control Logic/CTRL17
- J5 pad 20: /Control Logic/CTRL21 -> /Control Logic/CTRL26
- J5 pad 3: /Control Logic/CTRL2 -> /Control Logic/CTRL1
- J5 pad 4: /Control Logic/CTRL3 -> /Control Logic/CTRL18
- J5 pad 5: /Control Logic/CTRL4 -> /Control Logic/CTRL2
- J5 pad 6: /Control Logic/CTRL5 -> /Control Logic/CTRL19
- J5 pad 7: /Control Logic/CTRL6 -> /Control Logic/CTRL3
- J5 pad 8: /Control Logic/CTRL7 -> /Control Logic/CTRL20
- J5 pad 9: /Control Logic/CTRL8 -> /Control Logic/CTRL4
- U10 pad 1: unconnected-(U10-NC-Pad1) -> SYSDDIR
- U10 pad 10: /CPU/A15 -> +5V
- U10 pad 11: /CPU/A14 -> GND
- U10 pad 12: /CPU/A13 -> unconnected-(U10-XTAL2-Pad12)
- U10 pad 13: /Control Logic/MA13 -> CLK20
- U10 pad 14: /Control Logic/MA14 -> /SysIO/RX0
- U10 pad 15: /Control Logic/MA15 -> /SysIO/TX0
- U10 pad 16: GND -> /SysIO/RX1
- U10 pad 17: /Control Logic/MA16 -> /SysIO/TX1
- U10 pad 18: /Control Logic/MA17 -> SYSINT0
- U10 pad 19: /Control Logic/MA18 -> SYSINT1
- U10 pad 2: MMU_MAP13 -> ~{SYSDEN}
- U10 pad 20: /Control Logic/MA19 -> SYSINT2
- U10 pad 21: /Control Logic/MA20 -> SYSINTACK
- U10 pad 22: ~{MMU_RAM1_CE} -> /SysIO/KBCLK
- U10 pad 23: MMU_MAP7 -> /SysIO/KBDATA
- U10 pad 24: ~{MMU_RAM1_OE} -> /SysIO/TCK
- U10 pad 25: MMU_MAP8 -> /SysIO/TMS
- U10 pad 26: MMU_MAP6 -> /SysIO/TDO
- U10 pad 27: MMU_MAP5 -> /SysIO/TDI
- U10 pad 28: MMU_MAP10 -> Net-(U10-PC6)
- U10 pad 29: ~{MMU_RAM1_WE} -> Net-(U10-PC7)
- U10 pad 3: MMU_MAP11 -> SYSCMD
- U10 pad 31: MMU_MAP12 -> GND
- U10 pad 4: MMU_MAP9 -> BINTEN
- U10 pad 5: MMU_MAP4 -> /SysIO/~{SS}
- U10 pad 6: MMU_MAP3 -> /SysIO/MOSI
- U10 pad 7: MMU_MAP2 -> /SysIO/MISO
- U10 pad 8: MMU_MAP1 -> /SysIO/SCK
- U10 pad 9: MMU_MAP0 -> ~{CPU_RST}
- U11 pad 1: unconnected-(U11-NC-Pad1) -> SYSDDIR
- U11 pad 10: /CPU/A15 -> GND
- U11 pad 11: /CPU/A14 -> /CPU/D7
- U11 pad 12: /CPU/A13 -> /CPU/D6
- U11 pad 13: /Control Logic/MA21 -> /CPU/D5
- U11 pad 14: /Control Logic/MA22 -> /CPU/D4
- U11 pad 15: /Control Logic/MA23 -> /CPU/D3
- U11 pad 16: GND -> /CPU/D2
- U11 pad 17: /Control Logic/MA24 -> /CPU/D1
- U11 pad 18: /Control Logic/MA25 -> /CPU/D0
- U11 pad 19: MMU_MP_RD -> ~{SYSDEN}
- U11 pad 2: MMU_MAP13 -> Net-(U10-PA0)
- U11 pad 20: MMU_MP_WR -> +5V
- U11 pad 3: MMU_MAP11 -> Net-(U10-PA1)
- U11 pad 4: MMU_MAP9 -> Net-(U10-PA2)
- U11 pad 5: MMU_MAP4 -> Net-(U10-PA3)
- U11 pad 6: MMU_MAP3 -> Net-(U10-PA4)
- U11 pad 7: MMU_MAP2 -> Net-(U10-PA5)
- U11 pad 8: MMU_MAP1 -> Net-(U10-PA6)
- U11 pad 9: MMU_MAP0 -> Net-(U10-PA7)
- U3 pad 1: MMU_RAM1_DDIR -> MMU_RAM_DDIR
- U4 pad 1: MMU_RAM2_DDIR -> MMU_RAM_DDIR
- U7 pad 110: ~{MMU_RAM1_OE} -> ~{MMU_RAM1_WE}
- U7 pad 111: ~{MMU_RAM1_WE} -> ~{MMU_RAM2_CE}
- U7 pad 112: ~{MMU_RAM2_CE} -> ~{MMU_RAM2_WE}
- U7 pad 113: ~{MMU_RAM2_OE} -> MMU_RAM_DDIR
- U7 pad 115: ~{MMU_RAM2_WE} -> ~{MMU_RAM1_DE}
- U7 pad 116: MMU_RAM1_DDIR -> ~{MMU_RAM2_DE}
- U7 pad 117: ~{MMU_RAM1_DE} -> /Control Logic/CTRL4
- U7 pad 119: MMU_RAM2_DDIR -> /Control Logic/CTRL5
- U7 pad 120: ~{MMU_RAM2_DE} -> /Control Logic/CTRL6
- U7 pad 121: /Control Logic/CTRL4 -> /Control Logic/CTRL7
- U7 pad 124: /Control Logic/CTRL5 -> /Control Logic/CTRL8
- U7 pad 125: /Control Logic/CTRL6 -> /Control Logic/CTRL9
- U7 pad 69: MMU_MAP12 -> /Control Logic/CTRL25
- U7 pad 70: MMU_MAP13 -> /Control Logic/CTRL26
- U7 pad 86: /Control Logic/CTRL7 -> BINTEN
- U7 pad 87: /Control Logic/CTRL8 -> /Control Logic/CTRL10
- U7 pad 88: /Control Logic/CTRL9 -> /Control Logic/CTRL11
- U7 pad 91: /Control Logic/CTRL10 -> SYSDDIR
- U7 pad 92: /Control Logic/CTRL11 -> ~{SYSDEN}
- U7 pad 93: /Control Logic/CTRL12 -> SYSCMD
- U7 pad 94: /Control Logic/CTRL13 -> SYSINT0
- U7 pad 95: /Control Logic/CTRL14 -> SYSINT1
- U7 pad 96: /Control Logic/CTRL15 -> SYSINT2
- U7 pad 97: /Control Logic/CTRL16 -> SYSINTACK

Commit message: schematic updates
Parts:
- removed J10: SPI, Connector_PinSocket_2.54mm:PinSocket_2x03_P2.54mm_Vertical
- removed the J2 at (151.5, 120.9)
- removed the J5 at (218.6, 79.4)
- removed RN1: 10k, Resistor_THT:R_Array_SIP9
- added J8: SPI-SDCard, Connector_PinSocket_2.54mm:PinSocket_1x06_P2.54mm_Vertical, F.Cu at (256.5, 108.9)
- added R1: 10k, Resistor_SMD:R_0603_1608Metric_Pad0.98x0.95mm_HandSolder, F.Cu at (133.6, 21.8)
- added R10: 10k, Resistor_SMD:R_0603_1608Metric_Pad0.98x0.95mm_HandSolder, F.Cu at (138.0, 26.8)
- added R11: 10k, Resistor_SMD:R_0603_1608Metric_Pad0.98x0.95mm_HandSolder, F.Cu at (138.0, 29.3)
- added R12: 10k, Resistor_SMD:R_0603_1608Metric_Pad0.98x0.95mm_HandSolder, F.Cu at (138.0, 31.8)
- added R13: 10k, Resistor_SMD:R_0603_1608Metric_Pad0.98x0.95mm_HandSolder, F.Cu at (138.0, 34.3)
- added R14: 10k, Resistor_SMD:R_0603_1608Metric_Pad0.98x0.95mm_HandSolder, F.Cu at (138.0, 36.9)
- added R15: 10k, Resistor_SMD:R_0603_1608Metric_Pad0.98x0.95mm_HandSolder, F.Cu at (142.3, 21.8)
- added R16: 10k, Resistor_SMD:R_0603_1608Metric_Pad0.98x0.95mm_HandSolder, F.Cu at (142.3, 24.3)
- added R17: 10k, Resistor_SMD:R_0603_1608Metric_Pad0.98x0.95mm_HandSolder, F.Cu at (142.3, 26.8)
- added R18: 10k, Resistor_SMD:R_0603_1608Metric_Pad0.98x0.95mm_HandSolder, F.Cu at (142.3, 29.3)
- added R19: 10k, Resistor_SMD:R_0603_1608Metric_Pad0.98x0.95mm_HandSolder, F.Cu at (142.3, 31.8)
- added R2: 10k, Resistor_SMD:R_0603_1608Metric_Pad0.98x0.95mm_HandSolder, F.Cu at (133.6, 24.3)
- added R20: 10k, Resistor_SMD:R_0603_1608Metric_Pad0.98x0.95mm_HandSolder, F.Cu at (142.3, 34.3)
- added R21: 10k, Resistor_SMD:R_0603_1608Metric_Pad0.98x0.95mm_HandSolder, F.Cu at (142.3, 36.9)
- added R22: 10k, Resistor_SMD:R_0603_1608Metric_Pad0.98x0.95mm_HandSolder, F.Cu at (146.7, 21.8)
- added R23: 10k, Resistor_SMD:R_0603_1608Metric_Pad0.98x0.95mm_HandSolder, F.Cu at (146.7, 24.3)
- added R24: 10k, Resistor_SMD:R_0603_1608Metric_Pad0.98x0.95mm_HandSolder, F.Cu at (146.7, 26.8)
- added R25: 10k, Resistor_SMD:R_0603_1608Metric_Pad0.98x0.95mm_HandSolder, F.Cu at (146.7, 29.3)
- added R26: 10k, Resistor_SMD:R_0603_1608Metric_Pad0.98x0.95mm_HandSolder, F.Cu at (146.7, 31.8)
- added R27: 10k, Resistor_SMD:R_0603_1608Metric_Pad0.98x0.95mm_HandSolder, F.Cu at (226.3, 63.9)
- added R3: 10k, Resistor_SMD:R_0603_1608Metric_Pad0.98x0.95mm_HandSolder, F.Cu at (133.6, 26.8)
- added R35: 10k, Resistor_SMD:R_0603_1608Metric_Pad0.98x0.95mm_HandSolder, F.Cu at (219.9, 53.3)
- added R36: 10k, Resistor_SMD:R_0603_1608Metric_Pad0.98x0.95mm_HandSolder, F.Cu at (219.9, 60.9)
- added R37: 10k, Resistor_SMD:R_0603_1608Metric_Pad0.98x0.95mm_HandSolder, F.Cu at (219.9, 50.8)
- added R38: 10k, Resistor_SMD:R_0603_1608Metric_Pad0.98x0.95mm_HandSolder, F.Cu at (219.9, 55.8)
- added R39: 10k, Resistor_SMD:R_0603_1608Metric_Pad0.98x0.95mm_HandSolder, F.Cu at (219.9, 58.4)
- added R4: 10k, Resistor_SMD:R_0603_1608Metric_Pad0.98x0.95mm_HandSolder, F.Cu at (133.6, 29.3)
- added R40: 10k, Resistor_SMD:R_0603_1608Metric_Pad0.98x0.95mm_HandSolder, F.Cu at (219.9, 63.4)
- added R5: 10k, Resistor_SMD:R_0603_1608Metric_Pad0.98x0.95mm_HandSolder, F.Cu at (133.6, 31.8)
- added R6: 10k, Resistor_SMD:R_0603_1608Metric_Pad0.98x0.95mm_HandSolder, F.Cu at (133.6, 34.3)
- added R7: 10k, Resistor_SMD:R_0603_1608Metric_Pad0.98x0.95mm_HandSolder, F.Cu at (133.6, 36.9)
- added R8: 10k, Resistor_SMD:R_0603_1608Metric_Pad0.98x0.95mm_HandSolder, F.Cu at (138.0, 21.8)
- added R9: 10k, Resistor_SMD:R_0603_1608Metric_Pad0.98x0.95mm_HandSolder, F.Cu at (138.0, 24.3)
- added Y2: 32.768kHz, Crystal:Crystal_C26-LF_D2.1mm_L6.5mm_Horizontal, F.Cu at (225.5, 50.8)
- C1, C2, C3, C4, C5, C6: moved to B.Cu
- C10: renamed from C12; moved to B.Cu
- C11: renamed from C13; moved to B.Cu
- C12: renamed from C14; moved to B.Cu
- C13: renamed from C15; moved to B.Cu
- C14: renamed from C16; moved to B.Cu
- C15: renamed from C17; moved to B.Cu
- C16: renamed from C18; moved to B.Cu
- C17: renamed from C19; moved to B.Cu
- C7: renamed from C9; moved to B.Cu
- C8: renamed from C10; moved to B.Cu
- C9: renamed from C11; moved to B.Cu
- R28: renamed from R5; moved to B.Cu
- R29: renamed from R6; moved to B.Cu
- R30: renamed from R7; moved to B.Cu
- R31: renamed from R8; moved to B.Cu
- R32: renamed from R2; moved to B.Cu
- R33: renamed from R3; moved to B.Cu
- R34: renamed from R4; moved to B.Cu
- U11: renamed from U10; footprint Package_DIP:DIP-40_W15.24mm -> Package_DIP:DIP-40_W15.24mm_Socket_LongPads
- moved C21 151.2 mm to (129.3, 79.8)
- moved C22 151.2 mm to (129.3, 81.5)
- moved C5 101.2 mm to (208.6, 44.2)
- moved C6 101.2 mm to (208.6, 46.7)
- moved C16 78.0 mm to (169.6, 108.3), turned to 180 degrees
- moved J6 77.0 mm to (242.6, 101.4)
- moved J5 77.0 mm to (238.0, 101.4)
- moved J7 77.0 mm to (247.2, 101.4)
- moved C18 76.7 mm to (177.2, 80.0)
- moved C19 76.7 mm to (177.2, 91.5)
- moved C20 76.7 mm to (191.0, 80.0)
- moved C15 70.7 mm to (172.1, 115.7), turned to -90 degrees
- moved C7 70.0 mm to (173.0, 106.0), turned to 180 degrees
- moved R32 69.9 mm to (216.7, 89.3), turned to 180 degrees
- moved C17 69.9 mm to (216.7, 86.8), turned to 180 degrees
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- renumbered C20 to C18, C21 to C19, C24 to C20, C22 to C21, C23 to C22, C7 to C5, C8 to C6, J4 to J2, J6 to J4, J7 to J5, J8 to J6, J9 to J7, U3 to U1, U11 to U10, U1 to U2, U4 to U3, U2 to U4
Connections:
- J1 pad 15: /Expansion Bus/BB15 -> ~{BIACK}
- J1 pad 16: /Expansion Bus/BB16 -> BINTEN
- J1 pad 26: /Expansion Bus/BB26 -> BIRQ2
- J1 pad 27: /Expansion Bus/BB27 -> BIRQ1
- J1 pad 28: BINTEN -> BIRQ0
- J1 pad 32: /Expansion Bus/BA1 -> BA1
- J1 pad 4: BIRQ2 -> BB4
- J1 pad 6: /Expansion Bus/BB6 -> unconnected-(J1-DRQ2-Pad6)
- J1 pad 68: /Expansion Bus/BD6 -> BINTACK0
- J1 pad 69: /Expansion Bus/BD7 -> BINTACK1
- J1 pad 70: /Expansion Bus/BD8 -> BINTACK2
- J1 pad 71: /Expansion Bus/BD9 -> BINTACK3
- J1 pad 72: /Expansion Bus/BD10 -> BINTACK4
- J1 pad 73: /Expansion Bus/BD11 -> BINTACK5
- J1 pad 74: /Expansion Bus/BD12 -> BINTACK6
- J1 pad 75: /Expansion Bus/BD13 -> BINTACK7
- J1 pad 76: /Expansion Bus/BD14 -> unconnected-(J1-~{DACK7}-Pad76)
- J1 pad 77: /Expansion Bus/BD15 -> unconnected-(J1-DRQ7-Pad77)
- J1 pad 79: /Expansion Bus/BD17 -> unconnected-(J1-MASTER-Pad79)
- J1 pad 8: ~{BIACK} -> unconnected-(J1-UNUSED-Pad8)
- J1 pad 81: /Expansion Bus/BC1 -> BC1
- J1 pad 86: /Expansion Bus/BC6 -> BC6
- J1 pad 91: /Expansion Bus/BC11 -> BC11
- J1 pad 92: /Expansion Bus/BC12 -> BC12
- J1 pad 93: /Expansion Bus/BC13 -> BC13
- J1 pad 94: /Expansion Bus/BC14 -> BC14
- J1 pad 95: /Expansion Bus/BC15 -> BC15
- J1 pad 96: /Expansion Bus/BC16 -> BC16
- J1 pad 97: /Expansion Bus/BC17 -> BC17
- J1 pad 98: /Expansion Bus/BC18 -> BC18
- U1 pad 11: /Control Logic/MA20 -> /CPU/D7
- U1 pad 12: /Control Logic/MA19 -> /CPU/D6
- U1 pad 13: /Control Logic/MA18 -> /CPU/D5
- U1 pad 14: /Control Logic/MA17 -> /CPU/D4
- U1 pad 15: /Control Logic/MA16 -> /CPU/D3
- U1 pad 16: /Control Logic/MA15 -> /CPU/D2
- U1 pad 17: /Control Logic/MA14 -> /CPU/D1
- U1 pad 18: /Control Logic/MA13 -> /CPU/D0
- U1 pad 2: /CPU/D0 -> /Control Logic/MA13
- U1 pad 3: /CPU/D1 -> /Control Logic/MA14
- U1 pad 4: /CPU/D2 -> /Control Logic/MA15
- U1 pad 5: /CPU/D3 -> /Control Logic/MA16
- U1 pad 6: /CPU/D4 -> /Control Logic/MA17
- U1 pad 7: /CPU/D5 -> /Control Logic/MA18
- U1 pad 8: /CPU/D6 -> /Control Logic/MA19
- U1 pad 9: /CPU/D7 -> /Control Logic/MA20
- U3 pad 11: MMU_MP_EXE -> /CPU/D7
- U3 pad 12: MMU_MP_WR -> /CPU/D6
- U3 pad 13: MMU_MP_RD -> /CPU/D5
- U3 pad 14: /Control Logic/MA25 -> /CPU/D4
- U3 pad 15: /Control Logic/MA24 -> /CPU/D3
- U3 pad 16: /Control Logic/MA23 -> /CPU/D2
- U3 pad 17: /Control Logic/MA22 -> /CPU/D1
- U3 pad 18: /Control Logic/MA21 -> /CPU/D0
- U3 pad 2: /CPU/D0 -> /Control Logic/MA21
- U3 pad 3: /CPU/D1 -> /Control Logic/MA22
- U3 pad 4: /CPU/D2 -> /Control Logic/MA23
- U3 pad 5: /CPU/D3 -> /Control Logic/MA24
- U3 pad 6: /CPU/D4 -> /Control Logic/MA25
- U3 pad 7: /CPU/D5 -> MMU_MP_RD
- U3 pad 8: /CPU/D6 -> MMU_MP_WR
- U3 pad 9: /CPU/D7 -> MMU_MP_EXE
- U6 pad 31: ROM_WE# -> Net-(U6-WE#)
- U7 pad 100: /Control Logic/CTRL18 -> BINTACK1
- U7 pad 101: /Control Logic/CTRL19 -> BINTACK2
- U7 pad 102: /Control Logic/CTRL20 -> BINTACK3
- U7 pad 103: /Control Logic/CTRL21 -> BINTACK4
- U7 pad 104: /Control Logic/CTRL22 -> BINTACK5
- U7 pad 105: /Control Logic/CTRL23 -> BINTACK6
- U7 pad 107: /Control Logic/CTRL24 -> BINTACK7
- U7 pad 117: /Control Logic/CTRL4 -> BA1
- U7 pad 119: /Control Logic/CTRL5 -> BB4
- U7 pad 120: /Control Logic/CTRL6 -> BC15
- U7 pad 121: /Control Logic/CTRL7 -> BC16
- U7 pad 124: /Control Logic/CTRL8 -> BC17
- U7 pad 125: /Control Logic/CTRL9 -> BC18
- U7 pad 137: /Control Logic/CTRL0 -> BC11
- U7 pad 138: /Control Logic/CTRL1 -> BC12
- U7 pad 139: /Control Logic/CTRL2 -> BC13
- U7 pad 140: /Control Logic/CTRL3 -> BC14
- U7 pad 69: /Control Logic/CTRL25 -> BC1
- U7 pad 70: /Control Logic/CTRL26 -> BC6
- U7 pad 78: BIRQ2 -> BIRQ0
- U7 pad 79: BIRQ3 -> BIRQ1
- U7 pad 80: BIRQ4 -> BIRQ2
- U7 pad 81: BIRQ5 -> BIRQ3
- U7 pad 82: BIRQ6 -> BIRQ4
- U7 pad 83: BIRQ7 -> BIRQ5
- U7 pad 85: ~{BIACK} -> BIRQ6
- U7 pad 86: BINTEN -> BIRQ7
- U7 pad 87: /Control Logic/CTRL10 -> ~{BIACK}
- U7 pad 88: /Control Logic/CTRL11 -> BINTEN
- U7 pad 98: /Control Logic/CTRL17 -> BINTACK0
- Y1 pad 1: /CPU/CLK_E -> Net-(Y1-EN)
Routing:
- added copper zone on In2.Cu, net +5V
- added copper zone on In1.Cu, net GND
Other:
- board outline added: 222.4 x 105.4 mm
- board text added: "NOT ISA COMPATIBLE"
- board text removed: "https://jlcpcb.com/capabilities/pcb-capabilities"

Commit message: board
Parts:
- U1, U3: footprint Package_DIP:CERDIP-20_W7.62mm_SideBrazed_LongPads_Socket -> Package_DIP:DIP-20_W7.62mm_Socket_LongPads
- moved J3 51.3 mm to (260.6, 114.8)
- moved C1 44.0 mm to (167.0, 81.3)
- moved C2 44.0 mm to (167.0, 83.8)
- moved C21 44.0 mm to (173.1, 83.0)
- moved C22 44.0 mm to (173.1, 84.7)
- moved C3 44.0 mm to (167.0, 86.3)
- moved C4 44.0 mm to (167.0, 88.8)
- moved C5 44.0 mm to (167.0, 91.3)
- moved C6 44.0 mm to (167.0, 93.9)
- moved R29 36.6 mm to (222.5, 89.2)
- moved R30 36.6 mm to (222.5, 91.8)
- moved R31 36.6 mm to (222.5, 94.3)
- moved R28 36.6 mm to (222.5, 86.7)
- moved C14 25.7 mm to (196.9, 129.0)
- moved C10 25.7 mm to (215.5, 120.5)
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Connections:
- U11 pad 2: ~{SYSDEN} -> SYSCMD
- U11 pad 3: SYSCMD -> ~{SYSDEN}
