File: Main Board v2.0/Kicad/Main Board v2.0.kicad_pcb (KiCad board)
At the start: 4 copper layers, 222.4 x 105.4 mm, 85 parts, among them J1 Bus_ISA_16bit, J2 +3V3 Supply, J3 JTAG, J4 AVR-JTAG-10, J5 USART0, J6 USART1, J7 PS2KB, J8 SPI-SDCard, U1 74HCT245, U10 74HCT245, U11 ATmega1284-P, U2 GLT725608, U3 74HCT245, U4 GLT725608, U5 AS6C4008-55PCN, U6 AM29F040B, U7 XC95288XL-TQ144, U8 AP1117-33, U9 Z80CPU, Y1 20MHz, Y2 32.768kHz

Commit message: board update
Parts:
- removed the C5 at (167.0, 91.3)
- removed the C6 at (167.0, 93.9)
- added R41: 100R, Resistor_SMD:R_0603_1608Metric_Pad0.98x0.95mm_HandSolder, F.Cu at (166.7, 61.4)
- added SW1: Reset, Button_Switch_THT:SW_Tactile_SPST_Angled_PTS645Vx83-2LFS, F.Cu at (154.9, 70.0)
- C21, C22: footprint Capacitor_SMD:C_0201_0603Metric_Pad0.64x0.40mm_HandSolder -> Capacitor_SMD:C_0603_1608Metric_Pad1.08x0.95mm_HandSolder
- C5, C6, R27: moved to B.Cu
- Y1: footprint Oscillator:Oscillator_DIP-14 -> Oscillator:Oscillator_DIP-8_LargePads
- moved R27 86.4 mm to (141.1, 77.9), turned to -90 degrees
- moved R29 82.9 mm to (150.8, 47.8)
- moved R32 74.4 mm to (154.8, 48.0)
- moved R33 72.6 mm to (158.7, 48.3)
- moved C6 72.1 mm to (142.8, 76.1), turned to 90 degrees
- moved R34 71.5 mm to (162.2, 48.0)
- moved R28 68.4 mm to (166.0, 48.3)
- moved R30 68.3 mm to (169.8, 48.3)
- moved R31 67.1 mm to (173.6, 48.3)
- moved Y2 62.8 mm to (248.1, 109.5), turned to 180 degrees
- moved U1 61.9 mm to (198.2, 80.8)
- moved U3 57.6 mm to (211.4, 80.8)
- moved C18 57.1 mm to (223.6, 113.3)
- moved C19 56.9 mm to (223.9, 124.1)
- moved Y1 55.9 mm to (129.1, 126.5), turned to -90 degrees
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Connections:
- net Net-(U10-A0) renamed /SysIO/SYS_D0
- net Net-(U10-A1) renamed /SysIO/SYS_D1
- net Net-(U10-A2) renamed /SysIO/SYS_D2
- net Net-(U10-A3) renamed /SysIO/SYS_D3
- net Net-(U10-A4) renamed /SysIO/SYS_D4
- net Net-(U10-A5) renamed /SysIO/SYS_D5
- net Net-(U10-A6) renamed /SysIO/SYS_D6
- net Net-(U10-A7) renamed /SysIO/SYS_D7
- J1 pad 21: BIRQ7 -> BINTACK0
- J1 pad 22: BIRQ6 -> BINTACK1
- J1 pad 23: BIRQ5 -> BINTACK2
- J1 pad 50: /CPU/A12 -> /Control Logic/MA12
- J1 pad 6: unconnected-(J1-DRQ2-Pad6) -> BINTACK3
- J1 pad 65: /CPU/A13 -> /CPU/A12
- J1 pad 66: /CPU/A14 -> /CPU/A13
- J1 pad 67: /CPU/A15 -> /CPU/A14
- J1 pad 68: BINTACK0 -> /CPU/A15
- J1 pad 69: BINTACK1 -> unconnected-(J1-IRQ14-Pad69)
- J1 pad 70: BINTACK2 -> unconnected-(J1-~{DACK0}-Pad70)
- J1 pad 71: BINTACK3 -> unconnected-(J1-DRQ0-Pad71)
- J1 pad 72: BINTACK4 -> BINTACK5
- J1 pad 73: BINTACK5 -> BIRQ5
- J1 pad 75: BINTACK7 -> BIRQ6
- J1 pad 76: unconnected-(J1-~{DACK7}-Pad76) -> BINTACK7
- J1 pad 77: unconnected-(J1-DRQ7-Pad77) -> BIRQ7
- J1 pad 8: unconnected-(J1-UNUSED-Pad8) -> BINTACK4
- J1 pad 82: /Control Logic/MA23 -> BC2
- J1 pad 83: /Control Logic/MA22 -> BC3
- J1 pad 84: /Control Logic/MA21 -> /Control Logic/MA24
- J1 pad 85: /Control Logic/MA20 -> /Control Logic/MA23
- J1 pad 86: BC6 -> /Control Logic/MA22
- J1 pad 87: /Control Logic/MA25 -> /Control Logic/MA21
- J1 pad 88: /Control Logic/MA24 -> /Control Logic/MA20
- R1 pad 2: /Control Logic/MA14 -> /Control Logic/MA13
- R10 pad 2: /Control Logic/MA19 -> /Control Logic/MA18
- R11 pad 2: /Control Logic/MA21 -> /Control Logic/MA20
- R12 pad 2: /Control Logic/MA23 -> /Control Logic/MA22
- R13 pad 2: /Control Logic/MA25 -> /Control Logic/MA24
- R14 pad 1: /Control Logic/MA13 -> /Control Logic/MA12
- R15 pad 1: /Control Logic/MA15 -> /Control Logic/MA14
- R16 pad 1: /Control Logic/MA17 -> /Control Logic/MA16
- R17 pad 1: /Control Logic/MA19 -> /Control Logic/MA18
- R18 pad 1: /Control Logic/MA21 -> /Control Logic/MA20
- R19 pad 1: /Control Logic/MA23 -> /Control Logic/MA22
- R2 pad 2: /Control Logic/MA16 -> /Control Logic/MA15
- R20 pad 1: /Control Logic/MA25 -> /Control Logic/MA24
- R21 pad 1: /Control Logic/MA14 -> /Control Logic/MA13
- R22 pad 1: /Control Logic/MA16 -> /Control Logic/MA15
- R23 pad 1: /Control Logic/MA18 -> /Control Logic/MA17
- R24 pad 1: /Control Logic/MA20 -> /Control Logic/MA19
- R25 pad 1: /Control Logic/MA22 -> /Control Logic/MA21
- R26 pad 1: /Control Logic/MA24 -> /Control Logic/MA23
- R3 pad 2: /Control Logic/MA18 -> /Control Logic/MA17
- R4 pad 2: /Control Logic/MA20 -> /Control Logic/MA19
- R5 pad 2: /Control Logic/MA22 -> /Control Logic/MA21
- R6 pad 2: /Control Logic/MA24 -> /Control Logic/MA23
- R7 pad 2: /Control Logic/MA13 -> /Control Logic/MA12
- R8 pad 2: /Control Logic/MA15 -> /Control Logic/MA14
- R9 pad 2: /Control Logic/MA17 -> /Control Logic/MA16
- U1 pad 2: /Control Logic/MA13 -> /Control Logic/MA12
- U1 pad 3: /Control Logic/MA14 -> /Control Logic/MA13
- U1 pad 4: /Control Logic/MA15 -> /Control Logic/MA14
- U1 pad 5: /Control Logic/MA16 -> /Control Logic/MA15
- U1 pad 6: /Control Logic/MA17 -> /Control Logic/MA16
- U1 pad 7: /Control Logic/MA18 -> /Control Logic/MA17
- U1 pad 8: /Control Logic/MA19 -> /Control Logic/MA18
- U1 pad 9: /Control Logic/MA20 -> /Control Logic/MA19
- U2 pad 1: MMU_MAP11 -> MMU_MAP10
- U2 pad 10: /CPU/A13 -> /CPU/A12
- U2 pad 11: /Control Logic/MA13 -> /Control Logic/MA12
- U2 pad 12: /Control Logic/MA14 -> /Control Logic/MA13
- U2 pad 13: /Control Logic/MA15 -> /Control Logic/MA14
- U2 pad 15: /Control Logic/MA16 -> /Control Logic/MA15
- U2 pad 16: /Control Logic/MA17 -> /Control Logic/MA16
- U2 pad 17: /Control Logic/MA18 -> /Control Logic/MA17
- U2 pad 18: /Control Logic/MA19 -> /Control Logic/MA18
- U2 pad 19: /Control Logic/MA20 -> /Control Logic/MA19
- U2 pad 2: MMU_MAP9 -> MMU_MAP8
- U2 pad 21: MMU_MAP7 -> MMU_MAP6
- U2 pad 23: MMU_MAP8 -> MMU_MAP7
- U2 pad 24: MMU_MAP6 -> MMU_MAP5
- U2 pad 25: MMU_MAP5 -> MMU_MAP4
- U2 pad 26: MMU_MAP10 -> MMU_MAP9
- U2 pad 3: MMU_MAP4 -> MMU_MAP3
- U2 pad 4: MMU_MAP3 -> MMU_MAP2
- U2 pad 5: MMU_MAP2 -> MMU_MAP1
- U2 pad 6: MMU_MAP1 -> MMU_MAP0
- U2 pad 7: MMU_MAP0 -> /CPU/A15
- U2 pad 8: /CPU/A15 -> /CPU/A14
- U2 pad 9: /CPU/A14 -> /CPU/A13
- U3 pad 2: /Control Logic/MA21 -> /Control Logic/MA20
- U3 pad 3: /Control Logic/MA22 -> /Control Logic/MA21
- U3 pad 4: /Control Logic/MA23 -> /Control Logic/MA22
- U3 pad 5: /Control Logic/MA24 -> /Control Logic/MA23
- U3 pad 6: /Control Logic/MA25 -> /Control Logic/MA24
- U4 pad 1: MMU_MAP11 -> MMU_MAP10
- U4 pad 10: /CPU/A13 -> /CPU/A12
- U4 pad 11: /Control Logic/MA21 -> /Control Logic/MA20
- U4 pad 12: /Control Logic/MA22 -> /Control Logic/MA21
- U4 pad 13: /Control Logic/MA23 -> /Control Logic/MA22
- U4 pad 15: /Control Logic/MA24 -> /Control Logic/MA23
- U4 pad 16: /Control Logic/MA25 -> /Control Logic/MA24
- U4 pad 2: MMU_MAP9 -> MMU_MAP8
- U4 pad 21: MMU_MAP7 -> MMU_MAP6
- U4 pad 23: MMU_MAP8 -> MMU_MAP7
- U4 pad 24: MMU_MAP6 -> MMU_MAP5
- U4 pad 25: MMU_MAP5 -> MMU_MAP4
- U4 pad 26: MMU_MAP10 -> MMU_MAP9
- U4 pad 3: MMU_MAP4 -> MMU_MAP3
- U4 pad 4: MMU_MAP3 -> MMU_MAP2
- U4 pad 5: MMU_MAP2 -> MMU_MAP1
- U4 pad 6: MMU_MAP1 -> MMU_MAP0
- U4 pad 7: MMU_MAP0 -> /CPU/A15
- U4 pad 8: /CPU/A15 -> /CPU/A14
- U4 pad 9: /CPU/A14 -> /CPU/A13
- U5 pad 4: /CPU/A12 -> /Control Logic/MA12
- U6 pad 4: /CPU/A12 -> /Control Logic/MA12
- U7 pad 10: /CPU/D6 -> /CPU/A13
- U7 pad 100: BINTACK1 -> MMU_MAP4
- U7 pad 101: BINTACK2 -> MMU_MAP5
- U7 pad 102: BINTACK3 -> MMU_MAP6
- U7 pad 103: BINTACK4 -> MMU_MAP7
- U7 pad 104: BINTACK5 -> MMU_MAP8
- U7 pad 105: BINTACK6 -> MMU_MAP9
- U7 pad 106: ~{MMU_RAM1_CE} -> ~{MMU_RAM2_CE}
- U7 pad 107: BINTACK7 -> MMU_MAP10
- U7 pad 11: /CPU/D7 -> /CPU/A14
- U7 pad 110: ~{MMU_RAM1_WE} -> ~{MMU_RAM1_CE}
- U7 pad 111: ~{MMU_RAM2_CE} -> ~{MMU_RAM1_WE}
- U7 pad 112: ~{MMU_RAM2_WE} -> MMU_MP_RD
- U7 pad 113: MMU_RAM_DDIR -> MMU_MP_WR
- U7 pad 115: ~{MMU_RAM1_DE} -> MMU_MP_EXE
- U7 pad 116: ~{MMU_RAM2_DE} -> ~{RAM_CE}
- U7 pad 117: BA1 -> ~{ROM_CE}
- U7 pad 118: /Control Logic/MA20 -> BC3
- U7 pad 119: BB4 -> ~{CPU_HALT}
- U7 pad 12: ~{CPU_RST} -> /CPU/A15
- U7 pad 120: BC15 -> SYSDDIR
- U7 pad 121: BC16 -> ~{SYSDEN}
- U7 pad 124: BC17 -> SYSCMD
- U7 pad 125: BC18 -> SYSINTACK
- U7 pad 126: /Control Logic/MA21 -> SYSINT0
- U7 pad 128: /Control Logic/MA22 -> SYSINT1
- U7 pad 129: /Control Logic/MA23 -> SYSINT2
- U7 pad 13: ~{CPU_NMI} -> CLK20
- U7 pad 130: /Control Logic/MA24 -> ~{CPU_NMI}
- U7 pad 131: /Control Logic/MA25 -> ~{CPU_INT}
- U7 pad 132: MMU_MP_RD -> BC11
- U7 pad 133: MMU_MP_WR -> BC12
- U7 pad 134: MMU_MP_EXE -> BC13
- U7 pad 135: ~{ROM_CE} -> BC14
- U7 pad 136: ~{RAM_CE} -> BC15
- U7 pad 137: BC11 -> BC16
- U7 pad 138: BC12 -> BC17
- U7 pad 139: BC13 -> BC18
- U7 pad 14: ~{CPU_INT} -> ~{CPU_IORQ}
- U7 pad 140: BC14 -> BIRQ3
- U7 pad 142: ~{CPU_RFSH} -> ~{CPU_RD}
- U7 pad 143: ~{CPU_WAIT} -> ~{CPU_WR}
- U7 pad 15: ~{CPU_M1} -> ~{CPU_MREQ}
- U7 pad 16: /CPU/A0 -> BINTACK0
- U7 pad 17: /CPU/A1 -> BINTACK1
- U7 pad 19: /CPU/A2 -> /Control Logic/MA20
- U7 pad 2: /CPU/A15 -> BINTACK2
- U7 pad 20: /CPU/A3 -> /Control Logic/MA21
- U7 pad 21: /CPU/A4 -> /Control Logic/MA22
- U7 pad 22: /CPU/A5 -> /Control Logic/MA23
- U7 pad 23: /CPU/A6 -> /Control Logic/MA24
- U7 pad 24: /CPU/A7 -> BC1
- U7 pad 25: /CPU/A8 -> BC2
- U7 pad 26: /CPU/A9 -> /CPU/A0
- U7 pad 27: /CPU/A10 -> /CPU/A1
- U7 pad 28: /CPU/A11 -> /CPU/A2
- U7 pad 3: /CPU/D0 -> BINTACK3
- U7 pad 30: /CPU/A12 -> /CPU/A3
- U7 pad 31: /CPU/A13 -> /CPU/A4
- U7 pad 32: CLK20 -> BIRQ0
- U7 pad 33: ~{CPU_HALT} -> BIRQ1
- U7 pad 34: ~{CPU_RD} -> BIRQ2
- U7 pad 35: /CPU/A14 -> /CPU/A5
- U7 pad 38: ~{CPU_WR} -> /CPU/A6
- U7 pad 39: ~{CPU_MREQ} -> /CPU/A7
- U7 pad 4: /CPU/D1 -> BINTACK4
- U7 pad 40: ~{CPU_IORQ} -> /CPU/A8
- U7 pad 41: ~{CPU_BUSRQ} -> /CPU/A9
- U7 pad 43: ~{CPU_BUSACK} -> /CPU/A10
- U7 pad 44: /Control Logic/MA13 -> /CPU/A11
- U7 pad 45: /Control Logic/MA14 -> /Control Logic/MA12
- U7 pad 46: /Control Logic/MA15 -> /Control Logic/MA13
- U7 pad 48: /Control Logic/MA16 -> /Control Logic/MA14
- U7 pad 49: /Control Logic/MA17 -> /Control Logic/MA15
- U7 pad 5: /CPU/D2 -> BINTACK5
- U7 pad 50: /Control Logic/MA18 -> /Control Logic/MA16
- U7 pad 51: /Control Logic/MA19 -> /Control Logic/MA17
- U7 pad 52: MMU_MAP0 -> /Control Logic/MA18
- U7 pad 53: MMU_MAP1 -> /Control Logic/MA19
- U7 pad 54: MMU_MAP2 -> ~{CPU_M1}
- U7 pad 56: MMU_MAP3 -> ~{CPU_WAIT}
- U7 pad 57: MMU_MAP4 -> /CPU/D0
- U7 pad 58: MMU_MAP5 -> /CPU/D1
- U7 pad 59: MMU_MAP6 -> /CPU/D2
- U7 pad 6: /CPU/D3 -> BINTACK6
- U7 pad 60: MMU_MAP7 -> /CPU/D3
- U7 pad 61: MMU_MAP8 -> /CPU/D4
- U7 pad 64: MMU_MAP9 -> /CPU/D5
- U7 pad 66: MMU_MAP10 -> /CPU/D6
- U7 pad 68: MMU_MAP11 -> /CPU/D7
- U7 pad 69: BC1 -> BA1
- U7 pad 7: /CPU/D4 -> BINTACK7
- U7 pad 70: BC6 -> ~{CPU_RST}
- U7 pad 71: BCLK -> BB4
- U7 pad 74: ~{BIO_WR} -> ~{B8_MEM_WR}
- U7 pad 75: ~{BIO_RD} -> ~{B8_MEM_RD}
- U7 pad 76: ~{B8_MEM_WR} -> ~{BIO_WR}
- U7 pad 77: ~{B8_MEM_RD} -> ~{BIO_RD}
- U7 pad 78: BIRQ0 -> ~{BIACK}
- U7 pad 79: BIRQ1 -> BINTEN
- U7 pad 80: BIRQ2 -> ~{CPU_BUSRQ}
- U7 pad 81: BIRQ3 -> ~{CPU_BUSACK}
- U7 pad 82: BIRQ4 -> ~{CPU_RFSH}
- U7 pad 83: BIRQ5 -> BCLK
- U7 pad 85: BIRQ6 -> BIRQ7
- U7 pad 86: BIRQ7 -> BIRQ6
- U7 pad 87: ~{BIACK} -> BIRQ5
- U7 pad 88: BINTEN -> BIRQ4
- U7 pad 9: /CPU/D5 -> /CPU/A12
- U7 pad 91: SYSDDIR -> ~{MMU_RAM2_WE}
- U7 pad 92: ~{SYSDEN} -> MMU_RAM_DDIR
- U7 pad 93: SYSCMD -> ~{MMU_RAM1_DE}
- U7 pad 94: SYSINT0 -> ~{MMU_RAM2_DE}
- U7 pad 95: SYSINT1 -> MMU_MAP0
- U7 pad 96: SYSINT2 -> MMU_MAP1
- U7 pad 97: SYSINTACK -> MMU_MAP2
- U7 pad 98: BINTACK0 -> MMU_MAP3
- Y1 pad 8: CLK20 -> +5V
Routing:
- net /CPU/D3: track 0.00 -> 124.8 mm, vias 0 -> 3
- net /CPU/D5: track 0.00 -> 118.9 mm, vias 0 -> 4
- net /CPU/D4: track 0.00 -> 116.0 mm, vias 0 -> 3
- net /CPU/D6: track 0.00 -> 112.0 mm, vias 0 -> 4
- net /CPU/A15: track 0.00 -> 111.1 mm, vias 0 -> 4
- net /CPU/A14: track 0.00 -> 108.3 mm, vias 0 -> 4
- net /CPU/A13: track 0.00 -> 106.5 mm, vias 0 -> 4
- net /CPU/A12: track 0.00 -> 101.1 mm, vias 0 -> 2
- net /CPU/D7: track 0.00 -> 101.0 mm, vias 0 -> 2
- net /CPU/D2: track 0.00 -> 95.9 mm, vias 0 -> 3
- net /CPU/D1: track 0.00 -> 89.6 mm, vias 0 -> 2
- net /CPU/D0: track 0.00 -> 87.6 mm, vias 0 -> 2
- net /CPU/A11: track 0.00 -> 77.9 mm, vias 0 -> 1
- net ~{CPU_RD}: track 0.00 -> 71.3 mm, vias 0 -> 1
- net /Control Logic/MA15: track 0.00 -> 69.9 mm, vias 0 -> 4
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- added copper zone on In2.Cu, net +3V3
Other:
- board text added: "NOT ISA-BUS COMPATIBLE!"
- board text removed: "NOT ISA COMPATIBLE"

Commit message: board update
Parts:
- removed R28, R29, R30, R31: 100, Resistor_SMD:R_0603_1608Metric_Pad0.98x0.95mm_HandSolder
- C21, C22, R1, R10, R11, R12, R13, R14, R15, R16, R17, R18, R19, R2, R20, R21, R22, R23, R24, R25, R26, R3, R35, R36, R37, R38, R39, R4, R40, R41, R5, R6, R7, R8, R9: moved to B.Cu
- moved R32 134.2 mm to (266.5, 122.4), turned to -90 degrees
- moved R38 130.4 mm to (107.1, 117.6)
- moved R33 128.5 mm to (266.5, 118.1), turned to 90 degrees
- moved R39 127.9 mm to (107.1, 115.0)
- moved R34 122.9 mm to (266.5, 113.0), turned to 90 degrees
- moved R36 120.8 mm to (115.2, 117.6)
- moved R37 119.4 mm to (130.4, 126.2), turned to 180 degrees
- moved R40 118.4 mm to (115.2, 115.0), turned to 180 degrees
- moved C21 81.1 mm to (99.9, 102.3), turned to 180 degrees
- moved C22 78.0 mm to (130.4, 127.9), turned to 180 degrees
- moved C17 74.4 mm to (201.9, 116.3)
- moved R35 55.3 mm to (168.2, 69.3), turned to 180 degrees
- moved R1 40.4 mm to (216.1, 68.2), turned to -90 degrees
- moved R7 37.9 mm to (218.8, 68.2), turned to -90 degrees
- moved R8 34.5 mm to (213.3, 68.1), turned to -90 degrees
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Connections:
- net Net-(U11-PC6) renamed /SysIO/TOSC1
- net Net-(U11-PC7) renamed /SysIO/TOSC2
- J1 pad 32: BA1 -> ~{CPU_WAIT}
- J1 pad 4: BB4 -> ~{CPU_M1}
- J1 pad 41: ~{CPU_WAIT} -> /Control Logic/MA21
- J1 pad 42: ~{CPU_M1} -> /Control Logic/MA20
- J1 pad 84: /Control Logic/MA24 -> BC4
- J1 pad 85: /Control Logic/MA23 -> BC5
- J1 pad 86: /Control Logic/MA22 -> /Control Logic/MA24
- J1 pad 87: /Control Logic/MA21 -> /Control Logic/MA23
- J1 pad 88: /Control Logic/MA20 -> /Control Logic/MA22
- U7 pad 10: /CPU/A13 -> BC17
- U7 pad 11: /CPU/A14 -> BC16
- U7 pad 118: BC3 -> BINTACK0
- U7 pad 12: /CPU/A15 -> BC15
- U7 pad 122: Net-(U7-TDO) -> /Control Logic/TDO
- U7 pad 13: CLK20 -> BC14
- U7 pad 132: BC11 -> BINTACK1
- U7 pad 133: BC12 -> BIRQ0
- U7 pad 134: BC13 -> BIRQ1
- U7 pad 135: BC14 -> BIRQ2
- U7 pad 136: BC15 -> /CPU/A12
- U7 pad 137: BC16 -> /CPU/A13
- U7 pad 138: BC17 -> /CPU/A14
- U7 pad 139: BC18 -> /CPU/A15
- U7 pad 14: ~{CPU_IORQ} -> BC13
- U7 pad 142: ~{CPU_RD} -> ~{CPU_IORQ}
- U7 pad 143: ~{CPU_WR} -> ~{CPU_MREQ}
- U7 pad 15: ~{CPU_MREQ} -> BC12
- U7 pad 16: BINTACK0 -> BC11
- U7 pad 17: BINTACK1 -> ~{CPU_WR}
- U7 pad 19: /Control Logic/MA20 -> ~{CPU_RD}
- U7 pad 2: BINTACK2 -> BIRQ7
- U7 pad 20: /Control Logic/MA21 -> /Control Logic/MA22
- U7 pad 21: /Control Logic/MA22 -> /Control Logic/MA23
- U7 pad 22: /Control Logic/MA23 -> /Control Logic/MA24
- U7 pad 23: /Control Logic/MA24 -> BC5
- U7 pad 24: BC1 -> BC4
- U7 pad 25: BC2 -> BC3
- U7 pad 26: /CPU/A0 -> BC2
- U7 pad 27: /CPU/A1 -> BC1
- U7 pad 28: /CPU/A2 -> /CPU/A0
- U7 pad 3: BINTACK3 -> BINTACK7
- U7 pad 30: /CPU/A3 -> CLK20
- U7 pad 31: /CPU/A4 -> /CPU/A1
- U7 pad 32: BIRQ0 -> /CPU/A2
- U7 pad 33: BIRQ1 -> /CPU/A3
- U7 pad 34: BIRQ2 -> /CPU/A4
- U7 pad 4: BINTACK4 -> BIRQ6
- U7 pad 5: BINTACK5 -> BINTACK6
- U7 pad 54: ~{CPU_M1} -> /Control Logic/MA20
- U7 pad 56: ~{CPU_WAIT} -> /Control Logic/MA21
- U7 pad 6: BINTACK6 -> BIRQ5
- U7 pad 63: Net-(U7-TDI) -> /Control Logic/TDI
- U7 pad 65: Net-(U7-TMS) -> /Control Logic/TMS
- U7 pad 67: Net-(U7-TCK) -> /Control Logic/TCK
- U7 pad 69: BA1 -> ~{CPU_WAIT}
- U7 pad 7: BINTACK7 -> BINTACK5
- U7 pad 70: ~{CPU_RST} -> ~{CPU_M1}
- U7 pad 71: BB4 -> ~{CPU_RST}
- U7 pad 85: BIRQ7 -> BINTACK2
- U7 pad 86: BIRQ6 -> BINTACK3
- U7 pad 87: BIRQ5 -> BINTACK4
- U7 pad 9: /CPU/A12 -> BC18
Routing:
- net ~{CPU_RST}: track 0.00 -> 156.4 mm, vias 0 -> 2
- net ~{CPU_WR}: track 0.00 -> 132.8 mm, vias 0 -> 2
- net CLK20: track 0.00 -> 130.0 mm, vias 0 -> 4
- net ~{CPU_M1}: track 0.00 -> 116.3 mm, vias 0 -> 1
- net ~{CPU_WAIT}: track 0.00 -> 115.8 mm
- net /Control Logic/MA18: track 24.6 -> 138.2 mm, vias 0 -> 3
- net /Control Logic/MA16: track 24.0 -> 129.8 mm, vias 0 -> 2
- net /Control Logic/TDI: track 0.00 -> 104.7 mm, vias 0 -> 1
- net /Control Logic/TMS: track 0.00 -> 94.5 mm, vias 0 -> 1
- net /Control Logic/MA17: track 21.4 -> 115.2 mm, vias 0 -> 4
- net /Control Logic/TCK: track 0.00 -> 93.8 mm, vias 0 -> 1
- net ~{CPU_RFSH}: track 0.00 -> 87.6 mm
- net /Control Logic/MA21: track 0.00 -> 84.6 mm, vias 0 -> 1
- net /Control Logic/MA20: track 0.00 -> 84.0 mm, vias 0 -> 1
- net ~{CPU_RD}: track 71.3 -> 154.5 mm, vias 1 -> 3
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Other:
- board size 222.4 x 105.4 mm -> 172.7 x 83.9 mm
- board text added: "NOT A PC ISA CARD!"

Commit message: board progress
Routing:
- net /Control Logic/MA13: track 76.5 -> 65.0 mm
- net /Control Logic/MA14: track 81.2 -> 70.0 mm
- net /Control Logic/MA15: track 137.1 -> 126.3 mm
- net /Control Logic/MA16: track 129.8 -> 119.1 mm
- net /Control Logic/MA17: track 115.2 -> 105.0 mm
- net BINTACK2: track 30.3 -> 20.4 mm
- net /Control Logic/MA18: track 138.2 -> 128.4 mm
- net /Control Logic/MA19: track 50.7 -> 41.1 mm
- net /Control Logic/MA20: track 84.0 -> 74.9 mm
- net BIRQ4: track 29.3 -> 20.7 mm
- net /Control Logic/MA21: track 84.6 -> 76.3 mm
- net /CPU/D0: track 155.4 -> 147.2 mm
- net /CPU/D1: track 158.6 -> 150.9 mm
- net /CPU/D2: track 166.0 -> 158.6 mm
- net /Control Logic/MA12: track 83.1 -> 76.2 mm
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
Commit message: board progress
Parts:
- U1, U10, U3: footprint Package_DIP:DIP-20_W7.62mm_Socket_LongPads -> Library:DIP-20_W7.62mm_Socket_LongNarrowPads
- moved C21 17.5 mm to (91.5, 87.0)
- moved C6 17.5 mm to (134.4, 60.7)
- moved R27 17.5 mm to (132.7, 62.5)
- moved R39 17.5 mm to (98.7, 99.7)
- moved R40 17.5 mm to (106.9, 99.7)
- moved U6 17.5 mm to (121.5, 61.6)
- moved U9 17.5 mm to (94.8, 61.6)
- moved R36 17.5 mm to (106.9, 102.2)
- moved R38 17.5 mm to (98.7, 102.2)
- moved U5 16.3 mm to (154.0, 74.9)
- moved C5 16.3 mm to (161.5, 63.3)
- moved U2 15.5 mm to (174.2, 73.6)
- moved C2 15.5 mm to (175.1, 64.2)
- moved R1 15.4 mm to (216.1, 52.8)
- moved R10 15.4 mm to (202.1, 52.8)
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Connections:
- U7 pad 120: SYSDDIR -> ~{CPU_INT}
- U7 pad 121: ~{SYSDEN} -> ~{BIACK}
- U7 pad 124: SYSCMD -> ~{CPU_RFSH}
- U7 pad 125: SYSINTACK -> ~{CPU_BUSRQ}
- U7 pad 126: SYSINT0 -> BCLK
- U7 pad 128: SYSINT1 -> ~{CPU_BUSACK}
- U7 pad 129: SYSINT2 -> ~{CPU_NMI}
- U7 pad 130: ~{CPU_NMI} -> BINTACK1
- U7 pad 131: ~{CPU_INT} -> BINTACK2
- U7 pad 132: BINTACK1 -> BIRQ4
- U7 pad 133: BIRQ0 -> BIRQ3
- U7 pad 134: BIRQ1 -> BIRQ2
- U7 pad 135: BIRQ2 -> BIRQ1
- U7 pad 136: /CPU/A12 -> BIRQ0
- U7 pad 137: /CPU/A13 -> /CPU/A15
- U7 pad 139: /CPU/A15 -> /CPU/A13
- U7 pad 140: BIRQ3 -> A12
- U7 pad 74: ~{B8_MEM_WR} -> BINTACK4
- U7 pad 75: ~{B8_MEM_RD} -> BINTACK3
- U7 pad 76: ~{BIO_WR} -> ~{B8_MEM_WR}
- U7 pad 77: ~{BIO_RD} -> ~{B8_MEM_RD}
- U7 pad 78: ~{BIACK} -> ~{BIO_WR}
- U7 pad 79: BINTEN -> SYSINT2
- U7 pad 80: ~{CPU_BUSRQ} -> SYSINTACK
- U7 pad 81: ~{CPU_BUSACK} -> SYSINT1
- U7 pad 82: ~{CPU_RFSH} -> SYSCMD
- U7 pad 83: BCLK -> SYSINT0
- U7 pad 85: BINTACK2 -> BINTEN
- U7 pad 86: BINTACK3 -> SYSDDIR
- U7 pad 87: BINTACK4 -> ~{SYSDEN}
- U7 pad 88: BIRQ4 -> ~{BIO_RD}
- U9 pad 2: /CPU/A12 -> A12
Routing:
- net A12: track 0.00 -> 192.8 mm, vias 0 -> 3
- net /CPU/D6: track 171.1 -> 317.5 mm, vias 4 -> 7
- net /CPU/D2: track 158.6 -> 301.1 mm, vias 3 -> 5
- net /CPU/D0: track 147.2 -> 287.0 mm, vias 2 -> 4
- net /CPU/D5: track 175.8 -> 309.7 mm, vias 4 -> 6
- net /CPU/D1: track 150.9 -> 283.6 mm, vias 2 -> 4
- net /CPU/A12: track 129.0 -> 0.00 mm, vias 2 -> 0
- net CLK20: track 130.0 -> 250.1 mm, vias 4 -> 5
- net /CPU/D7: track 164.8 -> 274.1 mm, vias 2 -> 4
- net BINTEN: track 27.4 -> 129.7 mm, vias 0 -> 2
- net SYSCMD: track 0.00 -> 99.2 mm, vias 0 -> 1
- net SYSDDIR: track 0.00 -> 96.0 mm, vias 0 -> 1
- net /Control Logic/MA12: track 76.2 -> 163.4 mm, vias 2 -> 3
- net ~{SYSDEN}: track 0.00 -> 87.1 mm, vias 0 -> 1
- net /Control Logic/MA22: track 75.9 -> 161.5 mm, vias 1 -> 4
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Other:
- board size 172.7 x 83.9 mm -> 195.1 x 100.3 mm
