File: Main Board v2.0/Kicad/Main Board v2.0.kicad_pcb (KiCad board)
At the start: 4 copper layers, 195.1 x 100.3 mm, 81 parts, among them J1 Bus_ISA_16bit, J2 +3V3 Supply, J3 JTAG, J4 AVR-JTAG-10, J5 USART0, J6 USART1, J7 PS2KB, J8 SPI-SDCard, SW1 Reset, U1 74HCT245, U10 74HCT245, U11 ATmega1284-P, U2 GLT725608, U3 74HCT245, U4 GLT725608, U5 AS6C4008-55PCN, U6 AM29F040B, U7 XC95288XL-TQ144, U8 AP1117-33, U9 Z80CPU, Y1 20MHz, Y2 32.768kHz

Commit message: board rev a routed
Parts:
- moved C21 6.73 mm to (98.2, 87.0), turned to 0 degrees
- moved C1 3.88 mm to (205.8, 63.4)
- moved C3 3.81 mm to (219.0, 63.5)
- moved R1 2.29 mm to (218.8, 50.5)
- moved R10 2.29 mm to (193.7, 50.5)
- moved R11 2.29 mm to (190.9, 50.5)
- moved R12 2.29 mm to (188.1, 50.5)
- moved R13 2.29 mm to (185.3, 50.5)
- moved R14 2.29 mm to (218.8, 53.8)
- moved R16 2.29 mm to (213.3, 53.8)
- moved R17 2.29 mm to (210.5, 53.8)
- moved R18 2.29 mm to (207.7, 53.8)
- moved R19 2.29 mm to (204.9, 53.8)
- moved R2 2.29 mm to (216.1, 50.5)
- moved R20 2.29 mm to (202.1, 53.8)
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- renumbered R7 to R1, R5 to R10, R12 to R11, R6 to R12, R21 to R15, R15 to R16, R22 to R17, R16 to R18, R23 to R19, R1 to R2, R17 to R20, R24 to R21, R18 to R22, R25 to R23, R19 to R24, R26 to R25, R20 to R26, R35 to R27, R36 to R28, R38 to R29, R8 to R3, R39 to R30, R40 to R31, R41 to R32, R37 to R33, R27 to R34, R32 to R35, R33 to R36, R34 to R37, R2 to R4, R9 to R5, R3 to R6, R10 to R7, R4 to R8, R11 to R9
Connections:
- J1 pad 18: ~{CPU_BUSRQ} -> ~{BBUSRQ}
- J1 pad 91: BC11 -> unconnected-(J1-D8-Pad91)
- J1 pad 92: BC12 -> unconnected-(J1-D9-Pad92)
- U7 pad 10: BC17 -> BC18
- U7 pad 100: MMU_MAP4 -> MMU_MP_WR
- U7 pad 101: MMU_MAP5 -> ~{MMU_RAM1_WE}
- U7 pad 102: MMU_MAP6 -> ~{MMU_RAM2_WE}
- U7 pad 103: MMU_MAP7 -> MMU_MAP6
- U7 pad 104: MMU_MAP8 -> MMU_MAP7
- U7 pad 105: MMU_MAP9 -> ~{MMU_RAM1_CE}
- U7 pad 106: ~{MMU_RAM2_CE} -> MMU_MAP5
- U7 pad 107: MMU_MAP10 -> MMU_MAP4
- U7 pad 11: BC16 -> BC17
- U7 pad 110: ~{MMU_RAM1_CE} -> MMU_MAP9
- U7 pad 111: ~{MMU_RAM1_WE} -> MMU_MAP0
- U7 pad 112: MMU_MP_RD -> MMU_MAP1
- U7 pad 113: MMU_MP_WR -> MMU_MAP2
- U7 pad 115: MMU_MP_EXE -> MMU_MAP3
- U7 pad 116: ~{RAM_CE} -> MMU_MAP8
- U7 pad 117: ~{ROM_CE} -> MMU_MAP10
- U7 pad 118: BINTACK0 -> ~{RAM_CE}
- U7 pad 119: ~{CPU_HALT} -> ~{CPU_NMI}
- U7 pad 12: BC15 -> BC16
- U7 pad 121: ~{BIACK} -> ~{ROM_CE}
- U7 pad 129: ~{CPU_NMI} -> ~{CPU_HALT}
- U7 pad 13: BC14 -> BC15
- U7 pad 14: BC13 -> BC14
- U7 pad 140: A12 -> /CPU/A12
- U7 pad 143: ~{CPU_MREQ} -> ~{CPU_RST}
- U7 pad 15: BC12 -> BC13
- U7 pad 16: BC11 -> ~{BBUSRQ}
- U7 pad 38: /CPU/A6 -> GND
- U7 pad 39: /CPU/A7 -> /CPU/A6
- U7 pad 40: /CPU/A8 -> /CPU/A7
- U7 pad 41: /CPU/A9 -> /CPU/A8
- U7 pad 43: /CPU/A10 -> /CPU/A9
- U7 pad 44: /CPU/A11 -> /CPU/A10
- U7 pad 45: /Control Logic/MA12 -> /CPU/A11
- U7 pad 46: /Control Logic/MA13 -> /Control Logic/MA12
- U7 pad 48: /Control Logic/MA14 -> /Control Logic/MA13
- U7 pad 49: /Control Logic/MA15 -> /Control Logic/MA14
- U7 pad 50: /Control Logic/MA16 -> /Control Logic/MA15
- U7 pad 51: /Control Logic/MA17 -> /Control Logic/MA16
- U7 pad 52: /Control Logic/MA18 -> /Control Logic/MA17
- U7 pad 53: /Control Logic/MA19 -> /Control Logic/MA18
- U7 pad 54: /Control Logic/MA20 -> /Control Logic/MA19
- U7 pad 56: /Control Logic/MA21 -> /Control Logic/MA20
- U7 pad 57: /CPU/D0 -> /Control Logic/MA21
- U7 pad 58: /CPU/D1 -> /CPU/D0
- U7 pad 59: /CPU/D2 -> /CPU/D1
- U7 pad 60: /CPU/D3 -> /CPU/D2
- U7 pad 61: /CPU/D4 -> /CPU/D3
- U7 pad 64: /CPU/D5 -> /CPU/D4
- U7 pad 66: /CPU/D6 -> /CPU/D5
- U7 pad 68: /CPU/D7 -> /CPU/D6
- U7 pad 69: ~{CPU_WAIT} -> /CPU/D7
- U7 pad 70: ~{CPU_M1} -> ~{CPU_WAIT}
- U7 pad 71: ~{CPU_RST} -> ~{CPU_M1}
- U7 pad 9: BC18 -> ~{CPU_MREQ}
- U7 pad 91: ~{MMU_RAM2_WE} -> ~{BIACK}
- U7 pad 92: MMU_RAM_DDIR -> BINTACK0
- U7 pad 95: MMU_MAP0 -> MMU_RAM_DDIR
- U7 pad 96: MMU_MAP1 -> MMU_MP_RD
- U7 pad 97: MMU_MAP2 -> MMU_MP_EXE
- U7 pad 98: MMU_MAP3 -> ~{MMU_RAM2_CE}
- U9 pad 2: A12 -> /CPU/A12
Routing:
- net /CPU/A12: track 0.00 -> 193.8 mm, vias 0 -> 3
- net A12: track 192.8 -> 0.00 mm, vias 3 -> 0
- net /Control Logic/MA19: track 41.1 -> 157.8 mm, vias 0 -> 4
- net /Control Logic/MA13: track 107.0 -> 212.2 mm, vias 4 -> 9
- net /Control Logic/MA23: track 74.1 -> 178.8 mm, vias 1 -> 6
- net /Control Logic/MA24: track 69.6 -> 172.0 mm, vias 2 -> 7
- net /CPU/A11: track 101.4 -> 200.2 mm, vias 1 -> 5
- net /Control Logic/TDO: track 0.00 -> 97.3 mm, vias 0 -> 1
- net /Control Logic/MA16: track 132.8 -> 224.8 mm, vias 2 -> 5
- net /Control Logic/MA17: track 115.4 -> 206.1 mm, vias 4 -> 6
- net /Control Logic/MA18: track 137.3 -> 224.0 mm, vias 3 -> 5
- net ~{CPU_RFSH}: track 85.7 -> 165.9 mm, vias 0 -> 3
- net /CPU/A10: track 93.2 -> 171.4 mm, vias 1 -> 5
- net /CPU/A8: track 95.8 -> 173.6 mm, vias 2 -> 4
- net ~{CPU_M1}: track 126.8 -> 202.1 mm, vias 1 -> 3
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- added copper zone on B.Cu, net GND
- added copper zone on F.Cu, net GND
Other:
- board size 195.1 x 100.3 mm -> 178.7 x 100.3 mm
- board text added: "+3V3"
- board text added: "0"
- board text added: "1"
- board text added: "Atmel/AVR"
- board text added: "CLK"
- board text added: "DAT"
- board text added: "KEYBOARD"
- board text added: "MA12"
- board text added: "MA24"
- board text added: "MISO"
- board text added: "MOSI"
- board text added: "R1"
- board text added: "R13"
- board text added: "R14"
- board text added: "R26"
- board text added: "RX"
- board text added: "SCK"
- board text added: "SERIAL"
- board text added: "SPI"
- board text added: "TX"
- board text added: "Xilinx"
- board text added: "Zalt II Canned Bytes 2026 Rev A"
- board text added: "~{SS}"

Commit message: final board
Parts:
- added C23: 100n, Capacitor_SMD:C_0603_1608Metric_Pad1.08x0.95mm_HandSolder, B.Cu at (244.7, 85.9)
- added C24: 100n, Capacitor_SMD:C_0603_1608Metric_Pad1.08x0.95mm_HandSolder, B.Cu at (231.3, 63.6)
- added C25: 100n, Capacitor_SMD:C_0603_1608Metric_Pad1.08x0.95mm_HandSolder, B.Cu at (250.0, 89.1)
Routing:
- net +5V: track 70.8 -> 84.5 mm, vias 24 -> 25
- net GND: track 104.8 -> 111.3 mm, vias 48 -> 308
- net /CPU/A3: track 139.6 -> 143.2 mm
- net /CPU/A15: track 222.3 -> 224.4 mm
- net ~{CPU_RD}: track 179.9 -> 178.1 mm
- net ~{CPU_WR}: track 167.1 -> 165.3 mm
- net /CPU/A13: track 216.1 -> 214.3 mm
- net CLK20: track 249.8 -> 251.4 mm
- net BINTACK1: track 45.2 -> 44.3 mm
- net BIRQ0: track 35.7 -> 36.6 mm
- net /CPU/A11: track 200.2 -> 199.4 mm
- net /Control Logic/MA15: track 217.6 -> 218.1 mm
