File: Main Board v2.0/Kicad/CPU.kicad_sch (KiCad schematic)
At the start: 4 parts, among them U1 Z80CPU, Y1 20MHz

Commit message: update
Other:
- moved on the sheet: U1, Y1

Commit message: schematic done*
Parts:
- added RN1: 10k, Resistor_THT:R_Array_SIP9, symbol Device:R_Network08
- C22: renamed from C1; footprint (none) -> Capacitor_SMD:C_0201_0603Metric_Pad0.64x0.40mm_HandSolder
- C23: renamed from C2; footprint (none) -> Capacitor_SMD:C_0201_0603Metric_Pad0.64x0.40mm_HandSolder
- U9: renamed from U1; footprint (none) -> Package_DIP:DIP-40_W15.24mm_Socket_LongPads
Connections:
- net +5V: now also RN1.1 (common); no longer Y1.1 (EN)
- net ~{BUSACK} renamed ~{CPU_BUSACK}
- net ~{BUSRQ} renamed ~{CPU_BUSRQ}
- net ~{CPU_BUSRQ}: now also RN1.6 (R5)
- net ~{HALT} renamed ~{CPU_HALT}
- net ~{INT} renamed ~{CPU_INT}
- net ~{CPU_INT}: now also RN1.4 (R3)
- net ~{IORQ} renamed ~{CPU_IORQ}
- net ~{MREQ} renamed ~{CPU_MREQ}
- net ~{NMI} renamed ~{CPU_NMI}
- net ~{CPU_NMI}: now also RN1.3 (R2)
- net ~{RD} renamed ~{CPU_RD}
- net ~{RESET} renamed ~{CPU_RST}
- net ~{CPU_RST}: now also RN1.2 (R1)
- net ~{RFSH} renamed ~{CPU_RFSH}
- net ~{WAIT} renamed ~{CPU_WAIT}
- net ~{CPU_WAIT}: now also RN1.5 (R4)
- net ~{WR} renamed ~{CPU_WR}
- net ~~{M1} renamed ~{CPU_M1}
- new net CLK_E: RN1.7 (R6), Y1.1 (EN)
- new net ROM_WE#: RN1.8 (R7)
- no-connect marks 0 -> 1
Other:
- note removed: "TODO: - Pullups on control inputs - Decouple Cs"

Commit message: board update
Parts:
- added C24: 100u, Capacitor_THT:CP_Radial_D10.0mm_P5.00mm, symbol Device:C_Polarized
- U9: footprint Package_DIP:DIP-40_W15.24mm_Socket_LongPads -> Socket:3M_Textool_240-1288-00-0602J_2x20_P2.54mm
Connections:
- net GND: now also C24.2
- net ~{CPU_RST}: now also C24.1
Other:
- note added: "Simple RC time for ~{RESET}"
Changed lines of the file:
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@@
 		(title "Zalt CPU and Clock")
+	)
+	(text "Simple RC time \nfor  ~{RESET}"
+		(exclude_from_sim no)
+		(at 148.844 158.496 0)
+		(effects
+			(font
+				(size 1.27 1.27)
+			)
+		)
 	)
 	(junction
@@
 	)
 	(junction
+		(at 129.54 138.43)
+		(diameter 0)
+		(color 0 0 0 0)
+	)
+	(junction
 		(at 129.54 54.61)
 		(diameter 0)
@@
 	(wire
 		(pts
+			(xy 129.54 138.43) (xy 129.54 160.02)
+		)
+		(stroke
+			(width 0)
+			(type default)
+		)
+	)
+	(wire
+		(pts
 			(xy 127 62.23) (xy 143.51 62.23)
 		)
@@
 		(pts
 			(xy 179.07 107.95) (xy 203.2 107.95)
+		)
+		(stroke
+			(width 0)
+			(type default)
+		)
+	)
+	(wire
+		(pts
+			(xy 129.54 167.64) (xy 129.54 172.72)
 		)
 		(stroke
@@
 	)
 	(hierarchical_label "A[0..15]"
-		(shape output)
+		(shape tri_state)
 		(at 220.98 41.91 0)
 		(effects
@@
 			)
 		)
-		(property "Footprint" "Package_DIP:DIP-40_W15.24mm_Socket_LongPads"
+		(property "Footprint" "Socket:3M_Textool_240-1288-00-0602J_2x20_P2.54mm"
 			(at 161.29 74.93 0)
 			(hide yes)
@@
 					(unit 1)
 				)
+			)
+		)
+	)
+	(symbol
+		(lib_id "power:GND")
+		(at 129.54 172.72 0)
+		(unit 1)
+		(body_style 1)
+		(exclude_from_sim no)
+		(in_bom yes)
+		(on_board yes)
+		(in_pos_files yes)
+		(dnp no)
+		(fields_autoplaced yes)
+		(property "Reference" "#PWR087"
+			(at 129.54 179.07 0)
+			(hide yes)
+			(show_name no)
+			(do_not_autoplace no)
+			(effects
+				(font
+					(size 1.27 1.27)
+				)
+			)
+		)
+		(property "Value" "GND"
+			(at 129.54 177.8 0)
+			(show_name no)
+			(do_not_autoplace no)
+			(effects
+				(font
+					(size 1.27 1.27)
+				)
+			)
+		)
+		(property "Footprint" ""
+			(at 129.54 172.72 0)
+			(hide yes)
+			(show_name no)
+			(do_not_autoplace no)
+			(effects
+				(font
+					(size 1.27 1.27)
+				)
+			)
+		)
+		(property "Datasheet" ""
+			(at 129.54 172.72 0)
+			(hide yes)
+			(show_name no)
+			(do_not_autoplace no)
+			(effects
+				(font
+					(size 1.27 1.27)
+				)
+			)
+		)
+		(property "Description" "Power symbol creates a global label with name \"GND\" , ground"
+			(at 129.54 172.72 0)
+			(hide yes)
+			(show_name no)
+			(do_not_autoplace no)
+			(effects
+				(font
+					(size 1.27 1.27)
+				)
+			)
+		)
+		(pin "1"
+		)
+		(instances
+			(project "Main Board v2.0"
+				(path "/91a97de0-fe3a-4a53-b587-b32edd62d6f9/5629c61f-0e25-4cd4-88fe-4b15ad7083f0"
+					(reference "#PWR087")
+					(unit 1)
+				)
+			)
+		)
+	)
+	(symbol
+		(lib_id "Device:C_Polarized")
+		(at 129.54 163.83 0)
+		(unit 1)
+		(body_style 1)
+		(exclude_from_sim no)
+		(in_bom yes)
+		(on_board yes)
+		(in_pos_files yes)
+		(dnp no)
+		(fields_autoplaced yes)
+		(property "Reference" "C24"
+			(at 133.35 161.6709 0)
+			(show_name no)
+			(do_not_autoplace no)
+			(effects
+				(font
+					(size 1.27 1.27)
+				)
+				(justify left)
+			)
+		)
+		(property "Value" "100u"
+			(at 133.35 164.2109 0)
+			(show_name no)
+			(do_not_autoplace no)
+			(effects
+				(font
+					(size 1.27 1.27)
+				)
+				(justify left)
+			)
+		)
+		(property "Footprint" "Capacitor_THT:CP_Radial_D10.0mm_P5.00mm"
+			(at 130.5052 167.64 0)
+			(hide yes)
+			(show_name no)
+			(do_not_autoplace no)
+			(effects
+				(font
+					(size 1.27 1.27)
+				)
+			)
+		)
+		(property "Datasheet" ""
+			(at 129.54 163.83 0)
+			(hide yes)
+			(show_name no)
+			(do_not_autoplace no)
+			(effects
+				(font
+					(size 1.27 1.27)
+				)
+			)
+		)
+		(property "Description" "Polarized capacitor"
+			(at 129.54 163.83 0)
+			(hide yes)
+			(show_name no)
+			(do_not_autoplace no)
+			(effects
+				(font
+					(size 1.27 1.27)
+				)
+			)
+		)
+		(pin "1"
+		)
+		(pin "2"
+		)
+		(instances
+			(project "Main Board v2.0"
+				(path "/91a97de0-fe3a-4a53-b587-b32edd62d6f9/5629c61f-0e25-4cd4-88fe-4b15ad7083f0"
+					(reference "C24")
+					(unit 1)
+				)

Commit message: schematic update
Parts:
- C24: footprint Capacitor_THT:CP_Radial_D10.0mm_P5.00mm -> Capacitor_THT:CP_Radial_D8.0mm_P3.80mm
Changed lines of the file:
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@@
 			)
 		)
-		(property "Footprint" "Capacitor_THT:CP_Radial_D10.0mm_P5.00mm"
+		(property "Footprint" "Capacitor_THT:CP_Radial_D8.0mm_P3.80mm"
 			(at 130.5052 167.64 0)
 			(hide yes)

Commit message: schematic updates
Parts:
- removed RN1: 10k, Resistor_THT:R_Array_SIP9, symbol Device:R_Network08
- added R35, R36, R37, R38, R39, R40: 10k, Resistor_SMD:R_0603_1608Metric_Pad0.98x0.95mm_HandSolder, symbol Device:R_Small
- renumbered C24 to C20, C22 to C21, C23 to C22
Connections:
- net +5V: now also R35.1, R36.1, R37.1, R38.2, R39.2, R40.2
- net ~{CPU_BUSRQ}: now also R40.1
- net ~{CPU_INT}: now also R39.1
- net ~{CPU_NMI}: now also R38.1
- net ~{CPU_RST}: now also R35.2
- net ~{CPU_WAIT}: now also R36.2
- net CLK_E: no longer names the net of Y1.1 (EN)
- net CLK_E: now also R37.2
- no-connect marks 1 -> 0
Other:
- moved on the sheet: C20

Commit message: board update
Parts:
- added R41: 100R, Resistor_SMD:R_0603_1608Metric_Pad0.98x0.95mm_HandSolder, symbol Device:R_Small
- added SW1: Reset, Button_Switch_THT:SW_Tactile_SPST_Angled_PTS645Vx83-2LFS, symbol Switch:SW_Push
- C21, C22: footprint Capacitor_SMD:C_0201_0603Metric_Pad0.64x0.40mm_HandSolder -> Capacitor_SMD:C_0603_1608Metric_Pad1.08x0.95mm_HandSolder
- Y1: footprint Oscillator:Oscillator_DIP-14 -> Oscillator:Oscillator_DIP-8_LargePads
Connections:
- net +5V: now also Y1.8 (Vcc); no longer Y1.14 (Vcc)
- net CLK20: now also Y1.5 (OUT); no longer Y1.8 (OUT)
- net GND: now also Y1.4 (GND), SW1.1; no longer Y1.7 (GND)
- net ~{CPU_RST}: now also R41.2
- new net: R41.1, SW1.2

Commit message: board update
Parts:
- C20: KiLib_Generator (none) -> capacitor/THT/other
- C21, C22, R35, R36, R37, R38, R39, R40, R41: KiLib_Generator (none) -> SMD_2terminal_chip_molded
Changed lines of the file:
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@@
+			)
+		)
+		(property "KiLib_Generator" "SMD_2terminal_chip_molded"
+			(at 137.16 45.72 0)
+			(hide yes)
+			(show_name no)
+			(do_not_autoplace no)
+			(effects
+				(font
+					(size 1.27 1.27)
+				)
 			)
 		)
@@
 			)
 		)
+		(property "KiLib_Generator" "SMD_2terminal_chip_molded"
+			(at 132.08 127 0)
+			(hide yes)
+			(show_name no)
+			(do_not_autoplace no)
+			(effects
+				(font
+					(size 1.27 1.27)
+				)
+			)
+		)
 		(pin "1"
 		)
@@
 		)
 		(property "Description" "Resistor, small symbol"
+			(at 45.72 57.15 0)
+			(hide yes)
+			(show_name no)
+			(do_not_autoplace no)
+			(effects
+				(font
+					(size 1.27 1.27)
+				)
+			)
+		)
+		(property "KiLib_Generator" "SMD_2terminal_chip_molded"
 			(at 45.72 57.15 0)
 			(hide yes)
@@
 			)
 		)
+		(property "KiLib_Generator" "SMD_2terminal_chip_molded"
+			(at 100.33 43.18 0)
+			(hide yes)
+			(show_name no)
+			(do_not_autoplace no)
+			(effects
+				(font
+					(size 1.27 1.27)
+				)
+			)
+		)
 		(pin "1"
 		)
@@
 		)
 		(property "Description" "Resistor, small symbol"
+			(at 139.7 133.35 0)
+			(hide yes)
+			(show_name no)
+			(do_not_autoplace no)
+			(effects
+				(font
+					(size 1.27 1.27)
+				)
+			)
+		)
+		(property "KiLib_Generator" "SMD_2terminal_chip_molded"
 			(at 139.7 133.35 0)
 			(hide yes)
@@
 			)
 		)
+		(property "KiLib_Generator" "capacitor/THT/other"
+			(at 106.68 49.53 0)
+			(hide yes)
+			(show_name no)
+			(do_not_autoplace no)
+			(effects
+				(font
+					(size 1.27 1.27)
+				)
+			)
+		)
 		(pin "1"
 		)
@@
 			)
 		)
+		(property "KiLib_Generator" "SMD_2terminal_chip_molded"
+			(at 64.77 165.1 0)
+			(hide yes)
+			(show_name no)
+			(do_not_autoplace no)
+			(effects
+				(font
+					(size 1.27 1.27)
+				)
+			)
+		)
 		(pin "1"
 		)
@@
 			)
 		)
+		(property "KiLib_Generator" "SMD_2terminal_chip_molded"
+			(at 45.72 165.1 0)
+			(hide yes)
+			(show_name no)
+			(do_not_autoplace no)
+			(effects
+				(font
+					(size 1.27 1.27)
+				)
+			)
+		)
 		(pin "2"
 		)
@@
 			)
 		)
+		(property "KiLib_Generator" "SMD_2terminal_chip_molded"
+			(at 134.62 127 0)
+			(hide yes)
+			(show_name no)
+			(do_not_autoplace no)
+			(effects
+				(font
+					(size 1.27 1.27)
+				)
+			)
+		)
 		(pin "1"
 		)
@@
 			(at 129.54 45.72 0)
 			(hide yes)
+			(show_name no)
+			(do_not_autoplace no)
+			(effects
+				(font
+					(size 1.27 1.27)
+				)
+			)
+		)
+		(property "KiLib_Generator" "SMD_2terminal_chip_molded"
+			(at 129.54 45.72 0)
+			(hide yes)

Commit message: board rev a routed
Parts:
- renumbered R35 to R27, R36 to R28, R38 to R29, R39 to R30, R40 to R31, R41 to R32, R37 to R33
Changed lines of the file:
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@@
 		(in_pos_files yes)
 		(dnp no)
-		(property "Reference" "R36"
+		(property "Reference" "R28"
 			(at 138.43 44.45 0)
 			(show_name no)
@@
 			(project "Main Board v2.0"
 				(path "/91a97de0-fe3a-4a53-b587-b32edd62d6f9/5629c61f-0e25-4cd4-88fe-4b15ad7083f0"
-					(reference "R36")
+					(reference "R28")
 					(unit 1)
 				)
@@
 		(in_pos_files yes)
 		(dnp no)
-		(property "Reference" "R38"
+		(property "Reference" "R29"
 			(at 130.81 125.73 0)
 			(show_name no)
@@
 			(project "Main Board v2.0"
 				(path "/91a97de0-fe3a-4a53-b587-b32edd62d6f9/5629c61f-0e25-4cd4-88fe-4b15ad7083f0"
-					(reference "R38")
+					(reference "R29")
 					(unit 1)
 				)
@@
 		(in_pos_files yes)
 		(dnp no)
-		(property "Reference" "R37"
+		(property "Reference" "R33"
 			(at 46.99 55.88 0)
 			(show_name no)
@@
 			(project "Main Board v2.0"
 				(path "/91a97de0-fe3a-4a53-b587-b32edd62d6f9/5629c61f-0e25-4cd4-88fe-4b15ad7083f0"
-					(reference "R37")
+					(reference "R33")
 					(unit 1)
 				)
@@
 		(in_pos_files yes)
 		(dnp no)
-		(property "Reference" "R41"
+		(property "Reference" "R32"
 			(at 99.06 41.91 0)
 			(show_name no)
@@
 			(project "Main Board v2.0"
 				(path "/91a97de0-fe3a-4a53-b587-b32edd62d6f9/5629c61f-0e25-4cd4-88fe-4b15ad7083f0"
-					(reference "R41")
+					(reference "R32")
 					(unit 1)
 				)
@@
 		(in_pos_files yes)
 		(dnp no)
-		(property "Reference" "R40"
+		(property "Reference" "R31"
 			(at 140.97 132.08 0)
 			(show_name no)
@@
 			(project "Main Board v2.0"
 				(path "/91a97de0-fe3a-4a53-b587-b32edd62d6f9/5629c61f-0e25-4cd4-88fe-4b15ad7083f0"
-					(reference "R40")
+					(reference "R31")
 					(unit 1)
 				)
@@
 		(in_pos_files yes)
 		(dnp no)
-		(property "Reference" "R39"
+		(property "Reference" "R30"
 			(at 135.89 125.73 0)
 			(show_name no)
@@
 			(project "Main Board v2.0"
 				(path "/91a97de0-fe3a-4a53-b587-b32edd62d6f9/5629c61f-0e25-4cd4-88fe-4b15ad7083f0"
-					(reference "R39")
+					(reference "R30")
 					(unit 1)
 				)
@@
 		(in_pos_files yes)
 		(dnp no)
-		(property "Reference" "R35"
+		(property "Reference" "R27"
 			(at 130.81 44.45 0)
 			(show_name no)
@@
 			(project "Main Board v2.0"
 				(path "/91a97de0-fe3a-4a53-b587-b32edd62d6f9/5629c61f-0e25-4cd4-88fe-4b15ad7083f0"
-					(reference "R35")
-					(unit 1)
-				)
+					(reference "R27")
+					(unit 1)
+				)
