File: Main Board v2.0/Kicad/MMU.kicad_sch (KiCad schematic)
At the start: 34 parts, among them U1 74HCT245, U2 GLT725608, U3 74HCT245, U4 GLT725608

Commit message: board progress
Parts:
- U1, U3: footprint Package_DIP:DIP-20_W7.62mm_Socket_LongPads -> Library:DIP-20_W7.62mm_Socket_LongNarrowPads
Changed lines of the file:
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@@
 	)
 	(label "A12"
-		(at 68.58 43.18 0)
+		(at 72.39 43.18 180)
 		(effects
 			(font
 				(size 1.27 1.27)
 			)
-			(justify left bottom)
+			(justify right bottom)
 		)
 	)
@@
 			)
 		)
-		(property "Footprint" "Package_DIP:DIP-20_W7.62mm_Socket_LongPads"
+		(property "Footprint" "Library:DIP-20_W7.62mm_Socket_LongNarrowPads"
 			(at 194.31 123.19 0)
 			(hide yes)
@@
 			)
 		)
-		(property "Footprint" "Package_DIP:DIP-20_W7.62mm_Socket_LongPads"
+		(property "Footprint" "Library:DIP-20_W7.62mm_Socket_LongNarrowPads"
 			(at 194.31 55.88 0)
 			(hide yes)

Commit message: board rev a routed
Parts:
- renumbered R7 to R1, R5 to R10, R12 to R11, R6 to R12, R21 to R15, R15 to R16, R22 to R17, R16 to R18, R23 to R19, R1 to R2, R17 to R20, R24 to R21, R18 to R22, R25 to R23, R19 to R24, R26 to R25, R20 to R26, R8 to R3, R2 to R4, R9 to R5, R3 to R6, R10 to R7, R4 to R8, R11 to R9
Changed lines of the file:
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@@
 		(in_pos_files yes)
 		(dnp no)
-		(property "Reference" "R17"
+		(property "Reference" "R20"
 			(at 255.27 95.25 0)
 			(show_name no)
@@
 			(project "Main Board v2.0"
 				(path "/91a97de0-fe3a-4a53-b587-b32edd62d6f9/38464a8b-0df1-4971-a790-8d514365b55d"
-					(reference "R17")
+					(reference "R20")
 					(unit 1)
 				)
@@
 		(in_pos_files yes)
 		(dnp no)
-		(property "Reference" "R25"
+		(property "Reference" "R23"
 			(at 265.43 101.6 0)
 			(show_name no)
@@
 			(project "Main Board v2.0"
 				(path "/91a97de0-fe3a-4a53-b587-b32edd62d6f9/38464a8b-0df1-4971-a790-8d514365b55d"
-					(reference "R25")
+					(reference "R23")
 					(unit 1)
 				)
@@
 		(in_pos_files yes)
 		(dnp no)
-		(property "Reference" "R2"
+		(property "Reference" "R4"
 			(at 246.38 45.72 0)
 			(show_name no)
@@
 			(project "Main Board v2.0"
 				(path "/91a97de0-fe3a-4a53-b587-b32edd62d6f9/38464a8b-0df1-4971-a790-8d514365b55d"
-					(reference "R2")
+					(reference "R4")
 					(unit 1)
 				)
@@
 		(in_pos_files yes)
 		(dnp no)
-		(property "Reference" "R6"
+		(property "Reference" "R12"
 			(at 271.78 45.72 0)
 			(show_name no)
@@
 			(project "Main Board v2.0"
 				(path "/91a97de0-fe3a-4a53-b587-b32edd62d6f9/38464a8b-0df1-4971-a790-8d514365b55d"
-					(reference "R6")
+					(reference "R12")
 					(unit 1)
 				)
@@
 		(in_pos_files yes)
 		(dnp no)
-		(property "Reference" "R5"
+		(property "Reference" "R10"
 			(at 265.43 45.72 0)
 			(show_name no)
@@
 			(project "Main Board v2.0"
 				(path "/91a97de0-fe3a-4a53-b587-b32edd62d6f9/38464a8b-0df1-4971-a790-8d514365b55d"
-					(reference "R5")
+					(reference "R10")
 					(unit 1)
 				)
@@
 		(in_pos_files yes)
 		(dnp no)
-		(property "Reference" "R26"
+		(property "Reference" "R25"
 			(at 271.78 101.6 0)
 			(show_name no)
@@
 			(project "Main Board v2.0"
 				(path "/91a97de0-fe3a-4a53-b587-b32edd62d6f9/38464a8b-0df1-4971-a790-8d514365b55d"
-					(reference "R26")
+					(reference "R25")
 					(unit 1)
 				)
@@
 		(in_pos_files yes)
 		(dnp no)
-		(property "Reference" "R10"
+		(property "Reference" "R7"
 			(at 255.27 52.07 0)
 			(show_name no)
@@
 			(project "Main Board v2.0"
 				(path "/91a97de0-fe3a-4a53-b587-b32edd62d6f9/38464a8b-0df1-4971-a790-8d514365b55d"
-					(reference "R10")
+					(reference "R7")
 					(unit 1)
 				)
@@
 		(in_pos_files yes)
 		(dnp no)
-		(property "Reference" "R20"
+		(property "Reference" "R26"
 			(at 274.32 95.25 0)
 			(show_name no)
@@
 			(project "Main Board v2.0"
 				(path "/91a97de0-fe3a-4a53-b587-b32edd62d6f9/38464a8b-0df1-4971-a790-8d514365b55d"
-					(reference "R20")
+					(reference "R26")
 					(unit 1)
 				)
@@
 		(in_pos_files yes)
 		(dnp no)
-		(property "Reference" "R4"
+		(property "Reference" "R8"
 			(at 259.08 45.72 0)
 			(show_name no)
@@
 			(project "Main Board v2.0"
 				(path "/91a97de0-fe3a-4a53-b587-b32edd62d6f9/38464a8b-0df1-4971-a790-8d514365b55d"
-					(reference "R4")
+					(reference "R8")
 					(unit 1)
 				)
@@
 		(in_pos_files yes)
 		(dnp no)
-		(property "Reference" "R18"
+		(property "Reference" "R22"
 			(at 261.62 95.25 0)
 			(show_name no)
@@
 			(project "Main Board v2.0"
 				(path "/91a97de0-fe3a-4a53-b587-b32edd62d6f9/38464a8b-0df1-4971-a790-8d514365b55d"
-					(reference "R18")
+					(reference "R22")
 					(unit 1)
 				)
@@
 		(in_pos_files yes)
 		(dnp no)
-		(property "Reference" "R9"
+		(property "Reference" "R5"
 			(at 248.92 52.07 0)
 			(show_name no)
@@
 			(project "Main Board v2.0"
 				(path "/91a97de0-fe3a-4a53-b587-b32edd62d6f9/38464a8b-0df1-4971-a790-8d514365b55d"
-					(reference "R9")
+					(reference "R5")
 					(unit 1)
 				)
@@
 		(in_pos_files yes)
 		(dnp no)
-		(property "Reference" "R22"
+		(property "Reference" "R17"
 			(at 246.38 101.6 0)
 			(show_name no)
@@
 			(project "Main Board v2.0"
 				(path "/91a97de0-fe3a-4a53-b587-b32edd62d6f9/38464a8b-0df1-4971-a790-8d514365b55d"
-					(reference "R22")
+					(reference "R17")
 					(unit 1)
 				)
@@
 		(in_pos_files yes)
 		(dnp no)
-		(property "Reference" "R19"
+		(property "Reference" "R24"
 			(at 267.97 95.25 0)
 			(show_name no)
@@
 			(project "Main Board v2.0"
 				(path "/91a97de0-fe3a-4a53-b587-b32edd62d6f9/38464a8b-0df1-4971-a790-8d514365b55d"
-					(reference "R19")
+					(reference "R24")
 					(unit 1)
 				)
@@
 		(in_pos_files yes)
 		(dnp no)
-		(property "Reference" "R7"
+		(property "Reference" "R1"
 			(at 236.22 52.07 0)
 			(show_name no)
@@
 			(project "Main Board v2.0"
 				(path "/91a97de0-fe3a-4a53-b587-b32edd62d6f9/38464a8b-0df1-4971-a790-8d514365b55d"
-					(reference "R7")
+					(reference "R1")
 					(unit 1)
 				)
@@
 		(in_pos_files yes)
 		(dnp no)
-		(property "Reference" "R12"
+		(property "Reference" "R11"
 			(at 267.97 52.07 0)
 			(show_name no)
@@
 			(project "Main Board v2.0"
 				(path "/91a97de0-fe3a-4a53-b587-b32edd62d6f9/38464a8b-0df1-4971-a790-8d514365b55d"
-					(reference "R12")
+					(reference "R11")
 					(unit 1)
 				)
@@
 		(in_pos_files yes)
 		(dnp no)
-		(property "Reference" "R16"
+		(property "Reference" "R18"
 			(at 248.92 95.25 0)
 			(show_name no)
@@
 			(project "Main Board v2.0"
 				(path "/91a97de0-fe3a-4a53-b587-b32edd62d6f9/38464a8b-0df1-4971-a790-8d514365b55d"
-					(reference "R16")
+					(reference "R18")
 					(unit 1)
 				)
@@
 		(in_pos_files yes)
 		(dnp no)
-		(property "Reference" "R1"
+		(property "Reference" "R2"
 			(at 240.03 45.72 0)
 			(show_name no)
@@
 			(project "Main Board v2.0"
 				(path "/91a97de0-fe3a-4a53-b587-b32edd62d6f9/38464a8b-0df1-4971-a790-8d514365b55d"
-					(reference "R1")
+					(reference "R2")
 					(unit 1)
 				)
@@
 		(in_pos_files yes)
 		(dnp no)
-		(property "Reference" "R24"
+		(property "Reference" "R21"
 			(at 259.08 101.6 0)
 			(show_name no)
@@
 			(project "Main Board v2.0"
 				(path "/91a97de0-fe3a-4a53-b587-b32edd62d6f9/38464a8b-0df1-4971-a790-8d514365b55d"
-					(reference "R24")
+					(reference "R21")
 					(unit 1)
 				)
@@
 		(in_pos_files yes)
 		(dnp no)
-		(property "Reference" "R15"
+		(property "Reference" "R16"
 			(at 242.57 95.25 0)
 			(show_name no)
@@
 			(project "Main Board v2.0"
 				(path "/91a97de0-fe3a-4a53-b587-b32edd62d6f9/38464a8b-0df1-4971-a790-8d514365b55d"
-					(reference "R15")
+					(reference "R16")
 					(unit 1)
 				)
@@
 		(in_pos_files yes)
 		(dnp no)
-		(property "Reference" "R23"
+		(property "Reference" "R19"
 			(at 252.73 101.6 0)
 			(show_name no)
@@
 			(project "Main Board v2.0"
 				(path "/91a97de0-fe3a-4a53-b587-b32edd62d6f9/38464a8b-0df1-4971-a790-8d514365b55d"
-					(reference "R23")
+					(reference "R19")
 					(unit 1)
 				)
@@
 		(in_pos_files yes)
 		(dnp no)
-		(property "Reference" "R3"
+		(property "Reference" "R6"
 			(at 252.73 45.72 0)
 			(show_name no)
@@
 			(project "Main Board v2.0"
 				(path "/91a97de0-fe3a-4a53-b587-b32edd62d6f9/38464a8b-0df1-4971-a790-8d514365b55d"
-					(reference "R3")
+					(reference "R6")
 					(unit 1)
 				)
@@
 		(in_pos_files yes)
 		(dnp no)
-		(property "Reference" "R8"
+		(property "Reference" "R3"
 			(at 242.57 52.07 0)
 			(show_name no)
@@
 			(project "Main Board v2.0"
 				(path "/91a97de0-fe3a-4a53-b587-b32edd62d6f9/38464a8b-0df1-4971-a790-8d514365b55d"
-					(reference "R8")
+					(reference "R3")
 					(unit 1)
 				)
@@
 		(in_pos_files yes)
 		(dnp no)
-		(property "Reference" "R21"
+		(property "Reference" "R15"
 			(at 240.03 101.6 0)
 			(show_name no)
@@
 			(project "Main Board v2.0"
 				(path "/91a97de0-fe3a-4a53-b587-b32edd62d6f9/38464a8b-0df1-4971-a790-8d514365b55d"
-					(reference "R21")
+					(reference "R15")
 					(unit 1)
 				)
@@
 		(in_pos_files yes)
 		(dnp no)
-		(property "Reference" "R11"
+		(property "Reference" "R9"
 			(at 261.62 52.07 0)
 			(show_name no)
@@
 			(project "Main Board v2.0"
 				(path "/91a97de0-fe3a-4a53-b587-b32edd62d6f9/38464a8b-0df1-4971-a790-8d514365b55d"
-					(reference "R11")
+					(reference "R9")
 					(unit 1)
 				)
