File: Main Board v2.0/Kicad/SysIO.kicad_sch (KiCad schematic)
At the start: 8 parts, among them J10 SPI, J6 AVR-JTAG-10, J7 USART0, J8 USART1, J9 PS2KB, U10 ATmega1284-P, U11 74HCT245, Y2 32.768kHz

Commit message: docs
Other:
- note added: "Realtime Clock (no INT): - CMD: RTC-DATE - RD: Year (?) - RD: Month (1-12) - RD: Day (1-31) - CMD: RTC-TIME (can stop reading at any time) - RD: Hour (0-23) - RD: Minute (0-59) - RD: Second (0-59) BIOS Settings: - CMD: SETTING - WR: [address] (0-255) - RD: value / WR: value (0-255) Console: - CMD: CONSOLE-n (n:0-1) - WR: value (0-255) - output - (or) RD: value (0-255) - input, response to INT - S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"
- note removed: "Realtime Clock (no INT): - CMD: RTC-DATE - RD: Year (?) - RD: Month (1-12) - RD: Day (1-31) - CMD: RTC-TIME (can stop reading at any time) - RD: Hour (0-23) - RD: Minute (0-59) - RD: Second (0-59) - RD: Milli (0-99) BIOS Settings: - CMD: SETTING - WR: [address] (0-255) - RD: value / WR: value (0-255) Console: - CMD: CONSOLE-n (n:0-1) - WR: value (0-255) - output - (or) RD: value (0-255) - input, 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"
Changed lines of the file:
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@@
 		)
 	)
-	(text "Realtime Clock (no INT):\n- CMD: RTC-DATE\n	- RD: Year (?)\n	- RD: Month (1-12)\n	- RD: Day (1-31)\n\n- CMD: RTC-TIME (can stop reading at any time)\n	- RD: Hour (0-23)\n	- RD: Minute (0-59)\n	- RD: Second (0-59)\n	- RD: Milli (0-99)\n\nBIOS Settings:\n- CMD: SETTING\n	- WR: [address] (0-255)\n	- RD: value / WR: value (0-255)\n\nConsole:\n- CMD: CONSOLE-n (n:0-1)\n	- WR: value (0-255) - output\n	- (or) RD: value (0-255) - input, response to INT\n- STAT: OutputBufferEmpty, InputBufferFull\n- INT: receive input\n\nKeyboard (INT):\n- CMD: KEYBOARD (key-table values)\n	- RD: LSB\n	- RD: MSB\n- INT: receive input\n\nSystem-Timer:\n- INT every tick (100ms).\n\nProg Timers:\n- CMD: TIMER-n (n:0-?)\n	- WR: interval\n- INT every tick\n"
+	(text "Realtime Clock (no INT):\n- CMD: RTC-DATE\n	- RD: Year (?)\n	- RD: Month (1-12)\n	- RD: Day (1-31)\n\n- CMD: RTC-TIME (can stop reading at any time)\n	- RD: Hour (0-23)\n	- RD: Minute (0-59)\n	- RD: Second (0-59)\n\nBIOS Settings:\n- CMD: SETTING\n	- WR: [address] (0-255)\n	- RD: value / WR: value (0-255)\n\nConsole:\n- CMD: CONSOLE-n (n:0-1)\n	- WR: value (0-255) - output\n	- (or) RD: value (0-255) - input, response to INT\n- STAT: OutputBufferEmpty, InputBufferFull\n- INT: receive input\n\nKeyboard (INT):\n- CMD: KEYBOARD (key-table values)\n	- RD: LSB\n	- RD: MSB\n- INT: receive input\n\nSystem-Timer:\n- INT every tick (100ms).\n\nProg Timers:\n- CMD: TIMER-n (n:0-?)\n	- WR: interval\n- INT every tick\n"
 		(exclude_from_sim no)
 		(at 224.028 58.674 0)

Commit message: schematic updates
Parts:
- removed J10: SPI, Connector_PinSocket_2.54mm:PinSocket_2x03_P2.54mm_Vertical, symbol Connector_Generic:Conn_02x03_Odd_Even
- added J8: SPI-SDCard, Connector_PinSocket_2.54mm:PinSocket_1x06_P2.54mm_Vertical, symbol Connector_Generic:Conn_01x06
- U11: renamed from U10; footprint Package_DIP:DIP-40_W15.24mm -> Package_DIP:DIP-40_W15.24mm_Socket_LongPads
- Y2: footprint (none) -> Crystal:Crystal_C26-LF_D2.1mm_L6.5mm_Horizontal
- renumbered J6 to J4, J7 to J5, J8 to J6, J9 to J7, U11 to U10
Connections:
- net +5V: now also J8.2 (Pin_2)
- net GND: now also J8.1 (Pin_1)
- net MISO: now also J8.3 (Pin_3)
- net MOSI: now also J8.4 (Pin_4)
- net SCK: now also J8.5 (Pin_5)
- net SYSCMD: now also U11.2 (PB1); no longer U11.3 (PB2)
- net ~{SS}: now also J8.6 (Pin_6)
- net ~{SYSDEN}: now also U11.3 (PB2); no longer U11.2 (PB1)
Other:
- note added: "I2C"
- note added: "INT2"
- note added: "RD/~{WR}"
- note added: "SD-card module (24.2x42mm) SIL header: GND,VCC,MISO,MOSI,SCK,CS"
- note added: "Timer2=RTC"
- note added: "bdir"
- note added: "input"
- note added: "output"
- note added: "~{SYSDEN} (System Data Enable) is configured as INT2 on the MCU to be able to react as fast as possible to data exchange with the CPU."
- note removed: "Realtime Clock (no INT): - CMD: RTC-DATE - RD: Year (?) - RD: Month (1-12) - RD: Day (1-31) - CMD: RTC-TIME (can stop reading at any time) - RD: Hour (0-23) - RD: Minute (0-59) - RD: Second (0-59) BIOS Settings: - CMD: SETTING - WR: [address] (0-255) - RD: value / WR: value (0-255) Console: - CMD: CONSOLE-n (n:0-1) - WR: value (0-255) - output - (or) RD: value (0-255) - input, response to INT - S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"

Commit message: board update
Connections:
- net SYS_D7: now reaches U10.9 (A7), U11.33 (PA7)
- net SYS_D6: now reaches U10.8 (A6), U11.34 (PA6)
- net SYS_D5: now reaches U10.7 (A5), U11.35 (PA5)
- net SYS_D4: now reaches U10.6 (A4), U11.36 (PA4)
- net SYS_D3: now reaches U10.5 (A3), U11.37 (PA3)
- net SYS_D2: now reaches U10.4 (A2), U11.38 (PA2)
- net SYS_D1: now reaches U10.3 (A1), U11.39 (PA1)
- net SYS_D0: now reaches U10.2 (A0), U11.40 (PA0)
Changed lines of the file:
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@@
+		)
+	)
+	(label "SYS_D3"
+		(at 85.09 69.85 0)
+		(effects
+			(font
+				(size 1.27 1.27)
+			)
+			(justify left bottom)
+		)
+	)
+	(label "SYS_D1"
+		(at 85.09 64.77 0)
+		(effects
+			(font
+				(size 1.27 1.27)
+			)
+			(justify left bottom)
 		)
 	)
@@
 		)
 	)
+	(label "SYS_D2"
+		(at 85.09 67.31 0)
+		(effects
+			(font
+				(size 1.27 1.27)
+			)
+			(justify left bottom)
+		)
+	)
 	(label "TDI"
 		(at 93.98 120.65 180)
@@
 		)
 	)
+	(label "SYS_D4"
+		(at 85.09 72.39 0)
+		(effects
+			(font
+				(size 1.27 1.27)
+			)
+			(justify left bottom)
+		)
+	)
 	(label "D5"
 		(at 45.72 180.34 180)
@@
 		)
 	)
+	(label "SYS_D0"
+		(at 85.09 62.23 0)
+		(effects
+			(font
+				(size 1.27 1.27)
+			)
+			(justify left bottom)
+		)
+	)
 	(label "RX1"
 		(at 187.96 100.33 0)
@@
 		)
 	)
+	(label "SYS_D6"
+		(at 85.09 77.47 0)
+		(effects
+			(font
+				(size 1.27 1.27)
+			)
+			(justify left bottom)
+		)
+	)
 	(label "D0"
 		(at 45.72 167.64 180)
@@
 		(effects
 			(font
+				(size 1.27 1.27)
+			)
+			(justify left bottom)
+		)
+	)
+	(label "SYS_D7"
+		(at 85.09 80.01 0)
+		(effects
+			(font
+				(size 1.27 1.27)
+			)
+			(justify left bottom)
+		)
+	)
+	(label "SYS_D5"
+		(at 85.09 74.93 0)
+		(effects
+			(font

Commit message: board update
Parts:
- J4, J5, J6, J7, J8: KiLib_Generator (none) -> connector/pin_header_socket
- U10, U11: KiLib_Generator (none) -> package/DIP/legacy
- Y2: KiLib_Generator (none) -> crystal_resonator_oscillator
Connections:
- net TOSC1: now reaches U11.28 (PC6), Y2.1
- net TOSC2: now reaches U11.29 (PC7), Y2.2
Changed lines of the file:
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@@
+		)
+	)
+	(label "TOSC2"
+		(at 91.44 125.73 0)
+		(effects
+			(font
+				(size 1.27 1.27)
+			)
+			(justify left bottom)
 		)
 	)
@@
 			)
 			(justify right bottom)
+		)
+	)
+	(label "TOSC1"
+		(at 91.44 123.19 0)
+		(effects
+			(font
+				(size 1.27 1.27)
+			)
+			(justify left bottom)
 		)
 	)
@@
 			)
 		)
+		(property "KiLib_Generator" "connector/pin_header_socket"
+			(at 205.74 85.09 0)
+			(hide yes)
+			(show_name no)
+			(do_not_autoplace no)
+			(effects
+				(font
+					(size 1.27 1.27)
+				)
+			)
+		)
 		(pin "1"
 		)
@@
 			)
 		)
+		(property "KiLib_Generator" "crystal_resonator_oscillator"
+			(at 110.49 123.19 0)
+			(hide yes)
+			(show_name no)
+			(do_not_autoplace no)
+			(effects
+				(font
+					(size 1.27 1.27)
+				)
+			)
+		)
 		(pin "2"
 		)
@@
 			)
 		)
+		(property "KiLib_Generator" "package/DIP/legacy"
+			(at 66.04 105.41 0)
+			(hide yes)
+			(show_name no)
+			(do_not_autoplace no)
+			(effects
+				(font
+					(size 1.27 1.27)
+				)
+			)
+		)
 		(pin "5"
 		)
@@
 			)
 		)
+		(property "KiLib_Generator" "connector/pin_header_socket"
+			(at 180.34 46.99 0)
+			(hide yes)
+			(show_name no)
+			(do_not_autoplace no)
+			(effects
+				(font
+					(size 1.27 1.27)
+				)
+			)
+		)
 		(pin "2"
 		)
@@
 			)
 		)
+		(property "KiLib_Generator" "connector/pin_header_socket"
+			(at 205.74 134.62 0)
+			(hide yes)
+			(show_name no)
+			(do_not_autoplace no)
+			(effects
+				(font
+					(size 1.27 1.27)
+				)
+			)
+		)
 		(pin "1"
 		)
@@
 			)
 		)
+		(property "KiLib_Generator" "package/DIP/legacy"
+			(at 128.27 74.93 0)
+			(hide yes)
+			(show_name no)
+			(do_not_autoplace no)
+			(effects
+				(font
+					(size 1.27 1.27)
+				)
+			)
+		)
 		(pin "11"
 		)
@@
 			)
 		)
+		(property "KiLib_Generator" "connector/pin_header_socket"
+			(at 205.74 115.57 0)
+			(hide yes)
+			(show_name no)
+			(do_not_autoplace no)
+			(effects
+				(font
+					(size 1.27 1.27)
+				)
+			)
+		)
 		(pin "1"
 		)
@@
 			(at 205.74 100.33 0)
 			(hide yes)
+			(show_name no)
+			(do_not_autoplace no)
+			(effects
+				(font
+					(size 1.27 1.27)
+				)
+			)
+		)
+		(property "KiLib_Generator" "connector/pin_header_socket"
+			(at 205.74 100.33 0)
+			(hide yes)

Commit message: board progress
Parts:
- U10: footprint Package_DIP:DIP-20_W7.62mm_Socket_LongPads -> Library:DIP-20_W7.62mm_Socket_LongNarrowPads
Changed lines of the file:
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@@
 			)
 		)
-		(property "Footprint" "Package_DIP:DIP-20_W7.62mm_Socket_LongPads"
+		(property "Footprint" "Library:DIP-20_W7.62mm_Socket_LongNarrowPads"
 			(at 128.27 74.93 0)
 			(hide yes)

Commit message: final board
Parts:
- added C23, C24, C25: 100n, Capacitor_SMD:C_0603_1608Metric_Pad1.08x0.95mm_HandSolder, symbol Device:C
Connections:
- net +5V: now also C23.1, C24.1, C25.1
- net GND: now also C23.2, C24.2, C25.2
